File: Images/schematics/ad5754r-breakout/ad5754r-breakout.kicad_pcb (KiCad board)
At the start: 30 x 30 mm, 0 parts

Commit message: pcbs
Other:
- board text added: "AD5754BREZ Breakout"
- board text added: "MusicBrain v1.1"
- board text removed: "AD5754R Breakout"
- board text removed: "MusicBrain v1.0"
Changed lines of the file:
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@@
   (page A4)
   (title_block
-    (title "MusicBrain - AD5754R Minimal DAC Breakout Board")
-    (date "2026-06-06")
-    (rev "1.0")
+    (title "MusicBrain - AD5754BREZ Minimal DAC Breakout Board")
+    (date "2026-06-07")
+    (rev "1.1")
     (company "MusicBrain project")
-    (comment 1 "Quad 16-bit DAC, bipolar +/-5V, SSOP-28, SPI interface")
-    (comment 2 "ADR421 external 2.5V reference for 1V/oct pitch tracking")
+    (comment 1 "Quad 16-bit DAC, bipolar +/-5V, TSSOP-24, SPI interface")
+    (comment 2 "AD5754BREZ (non-R) requires ADR421 external 2.5V reference")
   )
   (layers
@@
   (net 7 "SDO")
   (net 8 "SYNC")
-  (net 9 "VOUT_A")
-  (net 10 "VOUT_B")
-  (net 11 "VOUT_C")
-  (net 12 "VOUT_D")
-  (net 13 "REF_2V5")
+  (net 9 "VOUTA")
+  (net 10 "VOUTB")
+  (net 11 "VOUTC")
+  (net 12 "VOUTD")
+  (net 13 "REFIN")
   (net 14 "CLR")
   (net 15 "LDAC")
-  (net 16 "RSET")
-  (net 17 "DCEN")
-  (net 18 "BIN_OFF")
+  (net 16 "BIN_2sCOMP")
   (net_class "Default" "This is the default net class."
     (clearance 0.2)
@@
   (gr_line (start 30 30) (end 0 30) (layer "Edge.Cuts") (width 0.05) (type solid))
   (gr_line (start 0 30) (end 0 0) (layer "Edge.Cuts") (width 0.05) (type solid))
-  (gr_text "AD5754R Breakout" (at 15 28) (layer "F.SilkS") (effects (font (size 1 1) (justify center))))
-  (gr_text "MusicBrain v1.0" (at 15 2) (layer "F.SilkS") (effects (font (size 0.8 0.8) (justify center))))
+  (gr_text "AD5754BREZ Breakout" (at 15 28) (layer "F.SilkS") (effects (font (size 1 1) (justify center))))
+  (gr_text "MusicBrain v1.1" (at 15 2) (layer "F.SilkS") (effects (font (size 0.8 0.8) (justify center))))
 )
