File: Images/schematics/ad5754r-breakout/ad5754r-breakout.kicad_pcb (KiCad board)
At the start: 30 x 30 mm, 0 parts

Commit message: kicad door fable
Parts:
- added C1: 10uF/25V, Capacitor_SMD:CP_Elec_4x5.3, F.Cu at (137.2, 111.5)
- added C2: 100nF, Capacitor_SMD:C_0805_2012Metric, F.Cu at (131.0, 111.5)
- added C3: 10uF/25V, Capacitor_SMD:CP_Elec_4x5.3, F.Cu at (113.5, 111.5)
- added C4: 100nF, Capacitor_SMD:C_0805_2012Metric, F.Cu at (119.0, 111.5)
- added C5: 100nF, Capacitor_SMD:C_0805_2012Metric, F.Cu at (131.5, 121.0)
- added C6: 100nF, Capacitor_SMD:C_0805_2012Metric, F.Cu at (132.5, 131.0)
- added C7: 100nF, Capacitor_SMD:C_0805_2012Metric, F.Cu at (120.0, 131.0)
- added C8: 10uF/25V, Capacitor_SMD:CP_Elec_4x5.3, F.Cu at (114.5, 131.0)
- added J1: SPI+Power, Connector_PinHeader_2.54mm:PinHeader_2x05_P2.54mm_Vertical, F.Cu at (105.5, 112.0)
- added J2: GND+DAC A-D, Connector_PinHeader_2.54mm:PinHeader_1x05_P2.54mm_Vertical, F.Cu at (145.5, 114.0)
- added R1: 10k, Resistor_SMD:R_0805_2012Metric, F.Cu at (119.0, 124.5)
- added R2: 100R, Resistor_SMD:R_0805_2012Metric, F.Cu at (139.5, 116.0)
- added R3: 100R, Resistor_SMD:R_0805_2012Metric, F.Cu at (139.5, 119.0)
- added R4: 100R, Resistor_SMD:R_0805_2012Metric, F.Cu at (139.5, 122.0)
- added R5: 100R, Resistor_SMD:R_0805_2012Metric, F.Cu at (139.5, 125.0)
- added U1: AD5754BREZ, Package_SO:HTSSOP-24-1EP_4.4x7.8mm_P0.65mm_EP3.2x5mm, F.Cu at (125.0, 118.0)
- added U2: ADR421, Package_SO:SOIC-8_3.9x4.9mm_P1.27mm, F.Cu at (126.0, 131.0)
Routing:
- added copper zone on B.Cu, net GND
- added copper zone on F.Cu, net GND
Other:
- board size 30 x 30 mm -> 50 x 35 mm
- copper layers 0 -> 2
- net class Default removed
- net class Power removed
- rule pad_to_mask_clearance: 0.04 -> 0
- board text added: "AD5754 DAC breakout rev 2.0"
- board text removed: "AD5754BREZ Breakout"
- board text removed: "MusicBrain v1.1"
