File: Images/schematics/ad5754r-breakout/ad5754r-breakout.kicad_pcb (KiCad board)
At the start: 2 copper layers, 50 x 35 mm, 17 parts, among them J1 SPI+Power, J2 GND+DAC A-D, U1 AD5754BREZ, U2 ADR421

Commit message: SPI-bus hardware: busspec, busboard, gate8-kaart; AD5754-breakout geroute
- doc/spi-bus-spec.md: leidende spec voor backplane + expansiekaarten
  (slot-pinout 2x10, geografische CS/IRQ, LDAC-buslijn, SPARE1=CONVST,
  ADC-keuze AD7606 naar teensy-eurorack van Nic Newdigate)
- musicbrain-busboard: Teensy 4.1 backplane, 6 slots + 2 IDC-hubs
  (sch ERC-schoon; PCB geplaatst met custom Teensy41-footprint,
  DRC 0 fouten, routing nog open)
- musicbrain-gate8: 8x gate out slotkaart met 74HCT595 @5V
  (sch + PCB volledig geroute, DRC 0/0)
- ad5754r-breakout: PCB volledig geroute (DRC 0 fouten, 0 unconnected);
  weerstanden 180 gedraaid, exposed pad via thermische via's aan -12V

Alles gevalideerd met kicad-cli 10 (ERC + netlist-check + DRC --refill-zones).

Co-Authored-By: Claude Fable 5 <noreply@anthropic.com>
Parts:
- turned R2 to 180 degrees
- turned R3 to 180 degrees
- turned R4 to 180 degrees
- turned R5 to 180 degrees
Routing:
- net +12V: track 0.00 -> 100.0 mm, vias 0 -> 4
- net -12V: track 0.00 -> 77.8 mm, vias 0 -> 5
- net +3V3: track 0.00 -> 58.4 mm, vias 0 -> 1
- net /SDO: track 0.00 -> 49.2 mm, vias 0 -> 1
- net /VOUTB: track 0.00 -> 28.5 mm
- net /VOUTA: track 0.00 -> 24.7 mm, vias 0 -> 2
- net /VREF: track 0.00 -> 21.0 mm
- net /SYNC: track 0.00 -> 20.4 mm
- net /VOUTD: track 0.00 -> 19.5 mm, vias 0 -> 2
- net /SDIN: track 0.00 -> 19.2 mm
- net /SCLK: track 0.00 -> 17.8 mm, vias 0 -> 1
- net /VOUTC: track 0.00 -> 17.1 mm
- net Net-(J2-Pin_5): track 0.00 -> 5.93 mm
- net Net-(U1-~{CLR}): track 0.00 -> 5.79 mm, vias 0 -> 2
- net Net-(J2-Pin_2): track 0.00 -> 5.63 mm
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