File: Images/schematics/ad5754r-breakout/ad5754r-breakout.kicad_sch (KiCad schematic)
At the start: 18 parts, among them J1 SPI+Power, J2 DAC Outputs, U1 AD5754R, U2 ADR421

Commit message: pcbs
Parts:
- removed R2: 6k8, Resistor_SMD:R_0805_2012Metric, symbol Device:R
- U1: value AD5754R -> AD5754BREZ; footprint Package_SO:SSOP-28_5.3x10.2mm_P0.65mm -> Package_SO:TSSOP-24_4.4x7.8mm_P0.65mm; symbol Custom:AD5754R -> Custom:AD5754BREZ
- renumbered R3 to R2, R4 to R3, R5 to R4, R6 to R5
Connections:
- no-connect marks 5 -> 9
Other:
- note added: "AD5754BREZ Minimal DAC Breakout"
- note added: "ADR421 Reference (MANDATORY): AD5754BREZ has NO internal reference ADR421 provides 2.5V ultra-precision (3 ppm/C) VOUT -> REFIN pin 17 Cannot omit U2 on this chip variant!"
- note added: "Control pins: LDAC -> GND (immediate update) CLR -> DVCC via 10k (no accidental clear) BIN/2sCOMP -> GND (twos complement coding) NC pins 2,6,12,13: leave unconnected"
- note added: "NOTE: This is the AD5754BREZ (TSSOP-24) NOT the AD5754R (SSOP-28). Pinout is different! See datasheet Table 5. No RSET, no DCEN, no BIN/OFF pin."
- note added: "Outputs: VOUTA-D -> 100R series -> header (short-circuit protection) +/-5V bipolar range (software config) 0x0000=-5V, 0x8000=0V, 0xFFFF=+5V"
- note added: "Power: AVDD = +12V (Eurorack) AVSS = -12V (Eurorack) DVCC = +3.3V (Teensy) All GND/DAC_GND/SIG_GND to unified ground plane Exposed paddle = AVSS (thermal)"
- note added: "Quad 16-bit DAC - Bipolar +/-5V mode TSSOP-24 package, SPI interface AD5754BREZ (non-R, no internal ref) Designed for JLCPCB PCBA assembly"
- note removed: "AD5754R Minimal DAC Breakout"
- note removed: "ADR421 Reference: 2.5V ultra-precision (3 ppm/C) Better than internal ref for 1V/oct Can omit U2 if internal ref is sufficient (then just add C6 on REFOUT pin)"
- note removed: "Control pins: LDAC -> DGND (immediate update) CLR -> DVCC via 10k (no accidental clear) DCEN -> DGND (daisy-chain off) BIN/OFF -> DGND (normal operation) RSET -> AGND via 6.8k"
- note removed: "NOTE: AI chat doc had WRONG pin numbers (described 24-pin package). AD5754R is SSOP-28. This schematic uses CORRECT pinout from datasheet Rev G."
- note removed: "Outputs: VOUT_A-D -> 100R series -> header (short-circuit protection) +/-5V bipolar range (software config) 0x0000=-5V, 0x8000=0V, 0xFFFF=+5V"
- note removed: "Power: AVDD = +12V (Eurorack) AVSS = -12V (Eurorack) DVCC = +3.3V (Teensy) All GND pins to unified ground plane"
- note removed: "Quad 16-bit DAC - Bipolar +/-5V mode SSOP-28 package, SPI interface Designed for JLCPCB PCBA assembly"
- title: MusicBrain - AD5754R Minimal DAC Breakout Board -> MusicBrain - AD5754BREZ Minimal DAC Breakout Board
