File: Images/schematics/ad5754r-breakout/ad5754r-breakout.kicad_sch (KiCad schematic)
At the start: 17 parts, among them J1 SPI+Power, J2 DAC Outputs, U1 AD5754BREZ, U2 ADR421

Commit message: kicad door fable
Parts:
- removed J2: DAC Outputs, Connector_PinHeader_2.54mm:PinHeader_1x04_P2.54mm_Vertical, symbol Connector_Generic:Conn_01x04
- added J2: GND+DAC A-D, Connector_PinHeader_2.54mm:PinHeader_1x05_P2.54mm_Vertical, symbol Connector_Generic:Conn_01x05
- C1, C3, C8: value 10uF -> 10uF/25V
- U1: footprint Package_SO:TSSOP-24_4.4x7.8mm_P0.65mm -> Package_SO:HTSSOP-24-1EP_4.4x7.8mm_P0.65mm_EP3.2x5mm
Connections:
- net SCLK: now also J1.5 (Pin_5), U1.8 (SCLK)
- net SDIN: now also J1.4 (Pin_4), U1.9 (SDIN)
- net SDO: now also J1.3 (Pin_3), U1.16 (SDO)
- net SYNC: now also J1.2 (Pin_2), U1.7 (~{SYNC})
- net VOUTA: now also R2.2, U1.3 (VOUTA)
- net VOUTB: now also R3.2, U1.4 (VOUTB)
- net VOUTC: now also R4.2, U1.23 (VOUTC)
- net VOUTD: now also R5.2, U1.22 (VOUTD)
- net -12V: now reaches U1.1 (AVSS)
- net -12V: now also C3.2 (-), C4.2, J1.9 (Pin_9), U1.25 (EPAD)
- net GND: now reaches U1.10 (~{LDAC})
- net GND: now also C1.2 (-), C2.2, C3.1 (+), C4.1, C5.2, C6.2, C7.2, C8.2 (-), J1.1 (Pin_1), J1.6 (Pin_6), J1.8 (Pin_8), U1.15 (GND), U1.18 (DAC_GND), U1.19 (DAC_GND), U1.20 (SIG_GND), U1.21 (SIG_GND), U2.4 (GND), J2.1 (Pin_1)
- net at U1.11 (~{CLR}): now also R1.2
- net +3V3: now reaches U1.14 (DVCC)
- net +3V3: now also C5.1, J1.7 (Pin_7), R1.1, U1.5 (BIN/2sCOMP)
- net VREF: now reaches U1.17 (REFIN)
- net VREF: now also C6.1, U2.8 (VOUT)
- net +12V: now reaches U1.24 (AVDD)
- net +12V: now also C1.1 (+), C2.1, C7.1, C8.1 (+), J1.10 (Pin_10), U2.2 (VIN)
- net at R2.1: now also J2.2 (Pin_2)
- net at R3.1: now also J2.3 (Pin_3)
- net at R4.1: now also J2.4 (Pin_4)
- net at R5.1: now also J2.5 (Pin_5)
Other:
- note added: "AD5754 Quad DAC Breakout - MusicBrain"
- note added: "Control pins: BIN/2sCOMP -> DVCC: OFFSET BINARY 0x0000 = -FS, 0x8000 = 0V, 0xFFFF = +FS (matches SPI-frame spec: 16-bit offset-binary) LDAC -> GND: output updates on SYNC rising edge CLR -> 10k pull-up to DVCC (no accidental clear)"
- note added: "J1 pinout (2x5 IDC, ribbon to controller): 1 GND 2 SYNC 3 SDO 4 SDIN 5 SCLK 6 GND 7 +3V3 8 GND 9 -12V 10 +12V"
- note added: "Outputs: VOUTA-D via 100R series to J2 (1x5): 1 GND, 2 OUTA, 3 OUTB, 4 OUTC, 5 OUTD (100R = short-circuit / cable protection)"
- note added: "Power: AVDD = +12V, AVSS = -12V (Eurorack) DVCC = +3V3 (logic side, Teensy/FPGA) Exposed pad (pin 25) tied to AVSS GND / DAC_GND / SIG_GND: one ground plane"
- note added: "Reference (MANDATORY): AD5754BREZ (non-R) has NO internal reference. ADR421 = 2.5V ultra-precision (3 ppm/C) -> REFIN. +/-5V range (software config) needs headroom: AVDD/AVSS >= +/-6.5V -> +/-12V is fine."
- note added: "SPI (mode 1: CPOL=0, CPHA=1; max 30 MHz): Teensy 4.1: SCLK=13(SCK), SDIN=11(MOSI), SDO=12(MISO), SYNC=10(CS) Data latched into DAC on SYNC rising edge"
- note added: "Supply decoupling (place at U1 pins on PCB)"
- note removed: "AD5754BREZ Minimal DAC Breakout"
- note removed: "ADR421 Reference (MANDATORY): AD5754BREZ has NO internal reference ADR421 provides 2.5V ultra-precision (3 ppm/C) VOUT -> REFIN pin 17 Cannot omit U2 on this chip variant!"
- note removed: "Control pins: LDAC -> GND (immediate update) CLR -> DVCC via 10k (no accidental clear) BIN/2sCOMP -> GND (twos complement coding) NC pins 2,6,12,13: leave unconnected"
- note removed: "NOTE: This is the AD5754BREZ (TSSOP-24) NOT the AD5754R (SSOP-28). Pinout is different! See datasheet Table 5. No RSET, no DCEN, no BIN/OFF pin."
- note removed: "Outputs: VOUTA-D -> 100R series -> header (short-circuit protection) +/-5V bipolar range (software config) 0x0000=-5V, 0x8000=0V, 0xFFFF=+5V"
- note removed: "Power: AVDD = +12V (Eurorack) AVSS = -12V (Eurorack) DVCC = +3.3V (Teensy) All GND/DAC_GND/SIG_GND to unified ground plane Exposed paddle = AVSS (thermal)"
- note removed: "Quad 16-bit DAC - Bipolar +/-5V mode TSSOP-24 package, SPI interface AD5754BREZ (non-R, no internal ref) Designed for JLCPCB PCBA assembly"
- note removed: "SPI (Teensy 4.1): SCLK -> Pin 13 (SCK) SDIN -> Pin 11 (MOSI) SDO -> Pin 12 (MISO) SYNC -> Pin 10 (CS) SPI Mode 1 (CPOL=0, CPHA=1)"
- title: MusicBrain - AD5754BREZ Minimal DAC Breakout Board -> MusicBrain - AD5754 Quad DAC Breakout
