File: Images/schematics/musicbrain-jack4/musicbrain-jack4.kicad_pcb (KiCad board)
At the start: 2 copper layers, 20 x 65 mm, 6 parts, among them J1 SOCKET-BACK, J2 PJ398SM, J3 PJ398SM, J4 PJ398SM, J5 PJ398SM

Commit message: Mechanica: L/B/H-assenstelsel + H=80mm-standaard (gedeelde bovenplaat)
- assenstelsel vastgelegd: L = busboard-lengte (kaartenrij), B = busboard-
  breedte (kaartvlakrichting), H = kaarthoogte boven het busboard
- H = 80 mm voor alle kaarten -> een vlakke bovenplaat draagt alle jacks,
  potmeters en encoders (GATE8 groeit in v1.1 van 60 naar 80)
- paneelconnector op de BOVENRAND, recht boven het slotcentrum (vervangt
  de eerdere 44mm-frontstandaard); jack-strips: header in het midden,
  strip loopt in B-richting en mag voor/achter de kaart uitsteken
- jack8/jack4 geregenereerd met gecentreerde header (DRC 0/0)

Co-Authored-By: Claude Fable 5 <noreply@anthropic.com>
Parts:
- moved J1 11.5 mm to (115.0, 126.2)
Routing:
- net /CH4: track 30.3 -> 18.8 mm
- net /CH1: track 21.1 -> 32.6 mm
- net /CH2: track 8.65 -> 20.1 mm
- net /CH3: track 17.8 -> 7.69 mm
Changed lines of the file:
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@@
   (footprint "MusicBrain:Header_1x06_backside"
     (layer "F.Cu")
-    (at 115 114.65)
+    (at 115 126.15)
     (descr "1x6 female socket - OP ACHTERZIJDE monteren (opening naar de kaart)")
     (property "Reference" "J1" (at 2.8 -2.2 0) (layer "F.SilkS")
@@
       (net 1 "GND"))
   )
-  (segment (start 115 117.19) (end 110.55 117.19) (width 0.25) (layer "F.Cu") (net 3))
-  (segment (start 110.55 117.19) (end 110.55 103.08) (width 0.25) (layer "F.Cu") (net 3))
-  (segment (start 110.55 103.08) (end 108 103.08) (width 0.25) (layer "F.Cu") (net 3))
-  (segment (start 115 119.73) (end 110.05 119.73) (width 0.25) (layer "F.Cu") (net 4))
-  (segment (start 110.05 119.73) (end 110.05 118.08) (width 0.25) (layer "F.Cu") (net 4))
-  (segment (start 110.05 118.08) (end 108 118.08) (width 0.25) (layer "F.Cu") (net 4))
-  (segment (start 115 122.27) (end 111.05 122.27) (width 0.25) (layer "F.Cu") (net 5))
-  (segment (start 111.05 122.27) (end 111.05 133.08) (width 0.25) (layer "F.Cu") (net 5))
-  (segment (start 111.05 133.08) (end 108 133.08) (width 0.25) (layer "F.Cu") (net 5))
-  (segment (start 115 124.81) (end 111.55 124.81) (width 0.25) (layer "F.Cu") (net 6))
-  (segment (start 111.55 124.81) (end 111.55 148.08) (width 0.25) (layer "F.Cu") (net 6))
+  (segment (start 115 128.69) (end 111.05 128.69) (width 0.25) (layer "F.Cu") (net 3))
+  (segment (start 111.05 128.69) (end 111.05 103.08) (width 0.25) (layer "F.Cu") (net 3))
+  (segment (start 111.05 103.08) (end 108 103.08) (width 0.25) (layer "F.Cu") (net 3))
+  (segment (start 115 131.23) (end 110.55 131.23) (width 0.25) (layer "F.Cu") (net 4))
+  (segment (start 110.55 131.23) (end 110.55 118.08) (width 0.25) (layer "F.Cu") (net 4))
+  (segment (start 110.55 118.08) (end 108 118.08) (width 0.25) (layer "F.Cu") (net 4))
+  (segment (start 115 133.77) (end 110.05 133.77) (width 0.25) (layer "F.Cu") (net 5))
+  (segment (start 110.05 133.77) (end 110.05 133.08) (width 0.25) (layer "F.Cu") (net 5))
+  (segment (start 110.05 133.08) (end 108 133.08) (width 0.25) (layer "F.Cu") (net 5))
+  (segment (start 115 136.31) (end 111.55 136.31) (width 0.25) (layer "F.Cu") (net 6))
+  (segment (start 111.55 136.31) (end 111.55 148.08) (width 0.25) (layer "F.Cu") (net 6))
   (segment (start 111.55 148.08) (end 108 148.08) (width 0.25) (layer "F.Cu") (net 6))
   (segment (start 108 111.38) (end 103.5 111.38) (width 0.3) (layer "F.Cu") (net 2))
