File: Images/schematics/musicbrain-jack8/musicbrain-jack8.kicad_pcb (KiCad board)
At the start: 2 copper layers, 20 x 125 mm, 10 parts, among them J1 SOCKET-BACK, J2 PJ398SM, J3 PJ398SM, J4 PJ398SM, J5 PJ398SM, J6 PJ398SM, J7 PJ398SM, J8 PJ398SM, J9 PJ398SM

Commit message: Mechanica: L/B/H-assenstelsel + H=80mm-standaard (gedeelde bovenplaat)
- assenstelsel vastgelegd: L = busboard-lengte (kaartenrij), B = busboard-
  breedte (kaartvlakrichting), H = kaarthoogte boven het busboard
- H = 80 mm voor alle kaarten -> een vlakke bovenplaat draagt alle jacks,
  potmeters en encoders (GATE8 groeit in v1.1 van 60 naar 80)
- paneelconnector op de BOVENRAND, recht boven het slotcentrum (vervangt
  de eerdere 44mm-frontstandaard); jack-strips: header in het midden,
  strip loopt in B-richting en mag voor/achter de kaart uitsteken
- jack8/jack4 geregenereerd met gecentreerde header (DRC 0/0)

Co-Authored-By: Claude Fable 5 <noreply@anthropic.com>
Parts:
- moved J1 18.5 mm to (115.0, 151.1)
Routing:
- net /CH8: track 25.2 -> 43.7 mm
- net /CH7: track 12.7 -> 31.2 mm
- net /CH5: track 26.2 -> 7.69 mm
- net /CH4: track 38.6 -> 20.1 mm
- net /CH3: track 51.1 -> 32.6 mm
- net /CH2: track 63.6 -> 45.1 mm
- net /CH1: track 76.0 -> 57.5 mm
- net /CH6: track 13.7 -> 18.8 mm
Changed lines of the file:
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@@
   (footprint "MusicBrain:Header_1x10_backside"
     (layer "F.Cu")
-    (at 115 169.57)
+    (at 115 151.07)
     (descr "1x10 female socket - OP ACHTERZIJDE monteren (opening naar de kaart)")
     (property "Reference" "J1" (at 2.8 -2.2 0) (layer "F.SilkS")
@@
       (net 1 "GND"))
   )
-  (segment (start 115 172.11) (end 112.55 172.11) (width 0.25) (layer "F.Cu") (net 3))
-  (segment (start 112.55 172.11) (end 112.55 103.08) (width 0.25) (layer "F.Cu") (net 3))
-  (segment (start 112.55 103.08) (end 108 103.08) (width 0.25) (layer "F.Cu") (net 3))
-  (segment (start 115 174.65) (end 112.05 174.65) (width 0.25) (layer "F.Cu") (net 4))
-  (segment (start 112.05 174.65) (end 112.05 118.08) (width 0.25) (layer "F.Cu") (net 4))
-  (segment (start 112.05 118.08) (end 108 118.08) (width 0.25) (layer "F.Cu") (net 4))
-  (segment (start 115 177.19) (end 111.55 177.19) (width 0.25) (layer "F.Cu") (net 5))
-  (segment (start 111.55 177.19) (end 111.55 133.08) (width 0.25) (layer "F.Cu") (net 5))
-  (segment (start 111.55 133.08) (end 108 133.08) (width 0.25) (layer "F.Cu") (net 5))
-  (segment (start 115 179.73) (end 111.05 179.73) (width 0.25) (layer "F.Cu") (net 6))
-  (segment (start 111.05 179.73) (end 111.05 148.08) (width 0.25) (layer "F.Cu") (net 6))
-  (segment (start 111.05 148.08) (end 108 148.08) (width 0.25) (layer "F.Cu") (net 6))
-  (segment (start 115 182.27) (end 110.55 182.27) (width 0.25) (layer "F.Cu") (net 7))
-  (segment (start 110.55 182.27) (end 110.55 163.08) (width 0.25) (layer "F.Cu") (net 7))
-  (segment (start 110.55 163.08) (end 108 163.08) (width 0.25) (layer "F.Cu") (net 7))
-  (segment (start 115 184.81) (end 110.05 184.81) (width 0.25) (layer "F.Cu") (net 8))
-  (segment (start 110.05 184.81) (end 110.05 178.08) (width 0.25) (layer "F.Cu") (net 8))
-  (segment (start 110.05 178.08) (end 108 178.08) (width 0.25) (layer "F.Cu") (net 8))
-  (segment (start 115 187.35) (end 113.05 187.35) (width 0.25) (layer "F.Cu") (net 9))
-  (segment (start 113.05 187.35) (end 113.05 193.08) (width 0.25) (layer "F.Cu") (net 9))
+  (segment (start 115 153.61) (end 112.05 153.61) (width 0.25) (layer "F.Cu") (net 3))
+  (segment (start 112.05 153.61) (end 112.05 103.08) (width 0.25) (layer "F.Cu") (net 3))
+  (segment (start 112.05 103.08) (end 108 103.08) (width 0.25) (layer "F.Cu") (net 3))
+  (segment (start 115 156.15) (end 111.55 156.15) (width 0.25) (layer "F.Cu") (net 4))
+  (segment (start 111.55 156.15) (end 111.55 118.08) (width 0.25) (layer "F.Cu") (net 4))
+  (segment (start 111.55 118.08) (end 108 118.08) (width 0.25) (layer "F.Cu") (net 4))
+  (segment (start 115 158.69) (end 111.05 158.69) (width 0.25) (layer "F.Cu") (net 5))
+  (segment (start 111.05 158.69) (end 111.05 133.08) (width 0.25) (layer "F.Cu") (net 5))
+  (segment (start 111.05 133.08) (end 108 133.08) (width 0.25) (layer "F.Cu") (net 5))
+  (segment (start 115 161.23) (end 110.55 161.23) (width 0.25) (layer "F.Cu") (net 6))
+  (segment (start 110.55 161.23) (end 110.55 148.08) (width 0.25) (layer "F.Cu") (net 6))
+  (segment (start 110.55 148.08) (end 108 148.08) (width 0.25) (layer "F.Cu") (net 6))
+  (segment (start 115 163.77) (end 110.05 163.77) (width 0.25) (layer "F.Cu") (net 7))
+  (segment (start 110.05 163.77) (end 110.05 163.08) (width 0.25) (layer "F.Cu") (net 7))
+  (segment (start 110.05 163.08) (end 108 163.08) (width 0.25) (layer "F.Cu") (net 7))
+  (segment (start 115 166.31) (end 112.55 166.31) (width 0.25) (layer "F.Cu") (net 8))
+  (segment (start 112.55 166.31) (end 112.55 178.08) (width 0.25) (layer "F.Cu") (net 8))
+  (segment (start 112.55 178.08) (end 108 178.08) (width 0.25) (layer "F.Cu") (net 8))
+  (segment (start 115 168.85) (end 113.05 168.85) (width 0.25) (layer "F.Cu") (net 9))
+  (segment (start 113.05 168.85) (end 113.05 193.08) (width 0.25) (layer "F.Cu") (net 9))
   (segment (start 113.05 193.08) (end 108 193.08) (width 0.25) (layer "F.Cu") (net 9))
-  (segment (start 115 189.89) (end 113.55 189.89) (width 0.25) (layer "F.Cu") (net 10))
-  (segment (start 113.55 189.89) (end 113.55 208.08) (width 0.25) (layer "F.Cu") (net 10))
+  (segment (start 115 171.39) (end 113.55 171.39) (width 0.25) (layer "F.Cu") (net 10))
+  (segment (start 113.55 171.39) (end 113.55 208.08) (width 0.25) (layer "F.Cu") (net 10))
   (segment (start 113.55 208.08) (end 108 208.08) (width 0.25) (layer "F.Cu") (net 10))
   (segment (start 108 111.38) (end 103.5 111.38) (width 0.3) (layer "F.Cu") (net 2))
