File: Images/schematics/musicbrain-gate8/musicbrain-gate8.kicad_sch (KiCad schematic)
At the start: 15 parts, among them J1 BUS, J2 GATES OUT, U1 74HCT595, U2 AMS1117-5.0

Commit message: GATE8 v1.1: H=80mm + haakse connectoren (bovenplaat-standaard)
- bord van 60x34 naar 35x80 mm (standaard-kaarthoogte H=80)
- J1 = haakse male 2x10 aan de onderrand (pennen het slot in),
  J2 = haakse male 1x10 aan de bovenrand, gecentreerd boven J1
- volledig opnieuw geroute: Q-netten als kruisingsvrije B.Cu-L-paden,
  SCLK/CS elk 1 B-hop, +5V-distributie via B-run; DRC 0/0, netlijst
  pad-voor-pad geverifieerd tegen het schema

Co-Authored-By: Claude Fable 5 <noreply@anthropic.com>
Parts:
- J1: footprint Connector_PinHeader_2.54mm:PinHeader_2x10_P2.54mm_Vertical -> Connector_PinHeader_2.54mm:PinHeader_2x10_P2.54mm_Horizontal
- J2: footprint Connector_PinHeader_2.54mm:PinHeader_1x10_P2.54mm_Vertical -> Connector_PinHeader_2.54mm:PinHeader_1x10_P2.54mm_Horizontal
Changed lines of the file:
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@@
     (property "Reference" "J1" (at 55 83.49 0) (effects (font (size 1.27 1.27))))
     (property "Value" "BUS" (at 55 116.51 0) (effects (font (size 1.27 1.27))))
-    (property "Footprint" "Connector_PinHeader_2.54mm:PinHeader_2x10_P2.54mm_Vertical" (at 55 100 0) (effects (font (size 1.27 1.27)) (hide yes)))
+    (property "Footprint" "Connector_PinHeader_2.54mm:PinHeader_2x10_P2.54mm_Horizontal" (at 55 100 0) (effects (font (size 1.27 1.27)) (hide yes)))
     (property "Datasheet" "" (at 55 100 0) (effects (font (size 1.27 1.27)) (hide yes)))
     (instances (project "musicbrain-gate8" (path "/d0000000-0000-4000-8000-000000000000" (reference "J1") (unit 1))))
@@
     (property "Reference" "J2" (at 165 81.03 0) (effects (font (size 1.27 1.27))))
     (property "Value" "GATES OUT" (at 165 111.51 0) (effects (font (size 1.27 1.27))))
-    (property "Footprint" "Connector_PinHeader_2.54mm:PinHeader_1x10_P2.54mm_Vertical" (at 165 95 0) (effects (font (size 1.27 1.27)) (hide yes)))
+    (property "Footprint" "Connector_PinHeader_2.54mm:PinHeader_1x10_P2.54mm_Horizontal" (at 165 95 0) (effects (font (size 1.27 1.27)) (hide yes)))
     (property "Datasheet" "" (at 165 95 0) (effects (font (size 1.27 1.27)) (hide yes)))
     (instances (project "musicbrain-gate8" (path "/d0000000-0000-4000-8000-000000000000" (reference "J2") (unit 1))))
