File: Images/schematics/musicbrain-busboard/musicbrain-busboard.kicad_sch (KiCad schematic)
At the start: 24 parts, among them J1 SLOT 1, J2 SLOT 2, J3 SLOT 3, J4 SLOT 4, J5 SLOT 5, J6 SLOT 6, J7 HUB 1, J8 HUB 2, J9 PWR IN, U1 Teensy 4.1, U2 R-78E5.0-0.5, U3 AMS1117-3.3

Commit message: Busboard v1.1: EXP-header, display-header (SPI1), Qwiic, M3-gaten
- J10 EXP (2x7): 8 vrije GPIO (D14-D17/D20-D23, analoog + Serial3/4/5)
  + 3V3/5V/GND; signalen via B.Cu-tussenrijlanen west van de Teensy
- J11 DISPLAY (1x9): eigen SPI1, pinvolgorde = ILI9341-module 1-op-1
  (CS=0, RESET=25, DC=24, MOSI1=26, SCK1=27, SDO nc)
- J12 QWIIC (1x4): GND/3V3/SDA/SCL op de bus-I2C, tussen slot 5 en 6
- 5x M3-montagegat voor standoffs (kast + bovenplaat)
- spec bijgewerkt: kaartstatussen v1.1, DAC8 bevestigd, RK097N-potten,
  display/EXP/Qwiic zoals gebouwd, mechanica-sectie 'dragen en geleiden'
  (slot + bovenplaat + standoffs; geen aparte printgeleiders nodig),
  encoderadvies Bourns PEC11R
- ERC 0, netlijst pad-voor-pad geverifieerd, DRC 0/0 (579 route-items)

Co-Authored-By: Claude Fable 5 <noreply@anthropic.com>
Parts:
- added J10: EXP, Connector_PinHeader_2.54mm:PinHeader_2x07_P2.54mm_Vertical, symbol Custom:Conn_02x07
- added J11: DISPLAY, Connector_PinHeader_2.54mm:PinHeader_1x09_P2.54mm_Vertical, symbol Custom:Conn_01x09
- added J12: QWIIC, Connector_PinHeader_2.54mm:PinHeader_1x04_P2.54mm_Vertical, symbol Custom:Conn_01x04
Connections:
- net +3V3: now also J10.1 (Pin_1), J11.1 (Pin_1), J11.8 (Pin_8), J12.2 (Pin_2)
- net +5V: now also J10.3 (Pin_3)
- net GND: now also J10.11 (Pin_11), J10.14 (Pin_14), J10.2 (Pin_2), J10.4 (Pin_4), J11.2 (Pin_2), J12.1 (Pin_1)
- net SCL: now also J12.4 (Pin_4)
- net SDA: now also J12.3 (Pin_3)
- net DISP_DC: now reaches U1.16 (24)
- net DISP_DC: now also J11.5 (Pin_5)
- net DISP_RST: now reaches U1.17 (25)
- net DISP_RST: now also J11.4 (Pin_4)
- net MOSI1: now reaches U1.18 (26)
- net MOSI1: now also J11.6 (Pin_6)
- net SCK1: now reaches U1.19 (27)
- net SCK1: now also J11.7 (Pin_7)
- net DISP_CS: now reaches U1.2 (0)
- net DISP_CS: now also J11.3 (Pin_3)
- net D14: now reaches U1.36 (14)
- net D14: now also J10.6 (Pin_6)
- net D15: now reaches U1.37 (15)
- net D15: now also J10.5 (Pin_5)
- net D16: now reaches U1.38 (16)
- net D16: now also J10.8 (Pin_8)
- net D17: now reaches U1.39 (17)
- net D17: now also J10.7 (Pin_7)
- net D20: now reaches U1.42 (20)
- net D20: now also J10.10 (Pin_10)
- net D21: now reaches U1.43 (21)
- net D21: now also J10.9 (Pin_9)
- net D22: now reaches U1.44 (22)
- net D22: now also J10.12 (Pin_12)
- net D23: now reaches U1.45 (23)
- net D23: now also J10.13 (Pin_13)
- no-connect marks 22 -> 10
