File: Images/schematics/musicbrain-dac8/musicbrain-dac8.kicad_pcb (KiCad board)
At the start: 2 copper layers, 50 x 80 mm, 25 parts, among them J1 BUS, J2 CV OUT, U1 AD5754BREZ, U2 AD5754BREZ, U3 ADR421

Commit message: DAC8-fix: correcte AD5754-pinout (~LDAC op pin 10, niet 12)
Bij het opzetten van de v2.1-check bleek de "zwevende LDAC" NIET in de
AD5754-breakout te zitten (die matcht Nick's bewezen ontwerp: pin 10 =
~LDAC, al aan GND; pin 12/13 = NC) maar in de deze sessie nieuw gemaakte
DAC8: daar was de AD5754-pinout verhaspeld (LDAC op pin 12 = NC-pad, echte
pin 10 aan GND). Gevolg: de bus-LDAC deed niets en de DAC updatete
transparant i.p.v. sample-synchroon.

- symbool + netmap gecorrigeerd tegen Nick's pinout: 5=BIN(+3V3),
  10=~LDAC(bus), 11=~CLR, 12/13=NC, 14=DVCC(+3V3), 15=DGND(GND)
- LDAC opnieuw geroute naar pin 10 via een trap-entry (CLR 0,6mm
  opgeschoven om ruimte te maken); U2-tak op F.Cu om de CS-B-hop te mijden
- ERC 0, netlijst pad-voor-pad geverifieerd, DRC 0/0; PDF's + fab herzien

De AD5754-breakout blijft ongewijzigd (was al correct).

Co-Authored-By: Claude Fable 5 <noreply@anthropic.com>
Connections:
- U1 pad 10: GND -> /LDAC
- U1 pad 12: /LDAC -> (no net)
- U2 pad 10: GND -> /LDAC
- U2 pad 12: /LDAC -> (no net)
Routing:
- net /LDAC: track 85.6 -> 92.0 mm
- net GND: track 5.80 -> 4.05 mm, vias 25 -> 23
- net /CLR: track 76.7 -> 75.5 mm
Changed lines of the file:
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@@
       (layers "F.Cu" "F.Mask" "F.Paste")
       (roundrect_rratio 0.25)
-      (net 4 "GND")
+      (net 9 "/LDAC")
     )
     (pad "11" smd roundrect
@@
       (layers "F.Cu" "F.Mask" "F.Paste")
       (roundrect_rratio 0.25)
-      (net 9 "/LDAC")
     )
     (pad "13" smd roundrect
@@
       (layers "F.Cu" "F.Mask" "F.Paste")
       (roundrect_rratio 0.25)
-      (net 4 "GND")
+      (net 9 "/LDAC")
     )
     (pad "11" smd roundrect
@@
       (layers "F.Cu" "F.Mask" "F.Paste")
       (roundrect_rratio 0.25)
-      (net 9 "/LDAC")
     )
     (pad "13" smd roundrect
@@
   (segment (start 107.7 170.2) (end 107.7 132.625) (width 0.25) (layer "F.Cu") (net 6))
   (segment (start 107.7 132.625) (end 110.625 132.625) (width 0.25) (layer "F.Cu") (net 6))
-  (segment (start 118.65 173.42) (end 118.65 167.3) (width 0.25) (layer "F.Cu") (net 9))
-  (segment (start 110.625 167.3) (end 122.1 167.3) (width 0.25) (layer "F.Cu") (net 9))
-  (segment (start 110.625 167.3) (end 110.625 134.575) (width 0.25) (layer "F.Cu") (net 9))
-  (segment (start 122.1 167.3) (end 122.1 163.6) (width 0.25) (layer "B.Cu") (net 9))
-  (segment (start 122.1 163.6) (end 122.1 134.575) (width 0.25) (layer "F.Cu") (net 9))
-  (segment (start 122.1 134.575) (end 124.625 134.575) (width 0.25) (layer "F.Cu") (net 9))
+  (segment (start 118.65 173.42) (end 118.65 166.5) (width 0.25) (layer "F.Cu") (net 9))
+  (segment (start 108.3 166.5) (end 118.65 166.5) (width 0.25) (layer "B.Cu") (net 9))
+  (segment (start 108.3 166.5) (end 108.3 133.275) (width 0.25) (layer "F.Cu") (net 9))
+  (segment (start 108.3 133.275) (end 110.625 133.275) (width 0.25) (layer "F.Cu") (net 9))
+  (segment (start 118.65 166.5) (end 121.4 166.5) (width 0.25) (layer "F.Cu") (net 9))
+  (segment (start 121.4 166.5) (end 121.4 133.275) (width 0.25) (layer "F.Cu") (net 9))
+  (segment (start 121.4 133.275) (end 124.625 133.275) (width 0.25) (layer "F.Cu") (net 9))
   (segment (start 121.19 173.42) (end 121.19 168.6) (width 0.25) (layer "F.Cu") (net 8))
   (segment (start 106.5 168.6) (end 121.19 168.6) (width 0.25) (layer "B.Cu") (net 8))
@@
   (segment (start 120 163.8) (end 120 131.325) (width 0.25) (layer "F.Cu") (net 8))
   (segment (start 120 131.325) (end 124.625 131.325) (width 0.25) (layer "F.Cu") (net 8))
-  (segment (start 108.3 162.4) (end 108.3 133.925) (width 0.25) (layer "F.Cu") (net 10))
-  (segment (start 108.3 133.925) (end 110.625 133.925) (width 0.25) (layer "F.Cu") (net 10))
-  (segment (start 108.3 162.4) (end 121.4 162.4) (width 0.25) (layer "B.Cu") (net 10))
-  (segment (start 121.4 162.4) (end 121.4 133.925) (width 0.25) (layer "F.Cu") (net 10))
-  (segment (start 121.4 133.925) (end 124.625 133.925) (width 0.25) (layer "F.Cu") (net 10))
+  (segment (start 108.9 162.4) (end 108.9 133.925) (width 0.25) (layer "F.Cu") (net 10))
+  (segment (start 108.9 133.925) (end 110.625 133.925) (width 0.25) (layer "F.Cu") (net 10))
+  (segment (start 108.9 162.4) (end 122 162.4) (width 0.25) (layer "B.Cu") (net 10))
+  (segment (start 122 162.4) (end 122 133.925) (width 0.25) (layer "F.Cu") (net 10))
+  (segment (start 122 133.925) (end 124.625 133.925) (width 0.25) (layer "F.Cu") (net 10))
   (segment (start 114.8 162.4) (end 114.8 161.3125) (width 0.25) (layer "F.Cu") (net 10))
   (segment (start 116.375 132.625) (end 118 132.625) (width 0.25) (layer "F.Cu") (net 11))
@@
   (segment (start 135.16 161.6) (end 144.4 161.6) (width 0.4) (layer "B.Cu") (net 2))
   (segment (start 144.4 161.6) (end 144.4 164.7) (width 0.4) (layer "F.Cu") (net 2))
-  (segment (start 110.625 133.275) (end 109.6 133.275) (width 0.25) (layer "F.Cu") (net 4))
-  (segment (start 124.625 133.275) (end 123.9 133.275) (width 0.25) (layer "F.Cu") (net 4))
   (segment (start 116.375 133.275) (end 118.3 133.275) (width 0.25) (layer "F.Cu") (net 4))
   (segment (start 130.375 133.275) (end 132.5 133.275) (width 0.25) (layer "F.Cu") (net 4))
@@
   (via (at 126.27 170.2) (size 0.5) (drill 0.3) (layers "F.Cu" "B.Cu") (net 6))
   (via (at 107.7 170.2) (size 0.5) (drill 0.3) (layers "F.Cu" "B.Cu") (net 6))
-  (via (at 122.1 167.3) (size 0.5) (drill 0.3) (layers "F.Cu" "B.Cu") (net 9))
-  (via (at 122.1 163.6) (size 0.5) (drill 0.3) (layers "F.Cu" "B.Cu") (net 9))
+  (via (at 118.65 166.5) (size 0.5) (drill 0.3) (layers "F.Cu" "B.Cu") (net 9))
+  (via (at 108.3 166.5) (size 0.5) (drill 0.3) (layers "F.Cu" "B.Cu") (net 9))
   (via (at 121.19 168.6) (size 0.5) (drill 0.3) (layers "F.Cu" "B.Cu") (net 8))
   (via (at 106.5 168.6) (size 0.5) (drill 0.3) (layers "F.Cu" "B.Cu") (net 8))
   (via (at 120 168.6) (size 0.5) (drill 0.3) (layers "F.Cu" "B.Cu") (net 8))
   (via (at 120 163.8) (size 0.5) (drill 0.3) (layers "F.Cu" "B.Cu") (net 8))
-  (via (at 108.3 162.4) (size 0.5) (drill 0.3) (layers "F.Cu" "B.Cu") (net 10))
-  (via (at 121.4 162.4) (size 0.5) (drill 0.3) (layers "F.Cu" "B.Cu") (net 10))
+  (via (at 108.9 162.4) (size 0.5) (drill 0.3) (layers "F.Cu" "B.Cu") (net 10))
+  (via (at 122 162.4) (size 0.5) (drill 0.3) (layers "F.Cu" "B.Cu") (net 10))
   (via (at 114.8 162.4) (size 0.5) (drill 0.3) (layers "F.Cu" "B.Cu") (net 10))
   (via (at 118 132.625) (size 0.5) (drill 0.3) (layers "F.Cu" "B.Cu") (net 11))
@@
   (via (at 117.05 121.1) (size 0.5) (drill 0.3) (layers "F.Cu" "B.Cu") (net 2))
   (via (at 144.4 161.6) (size 0.5) (drill 0.3) (layers "F.Cu" "B.Cu") (net 2))
-  (via (at 109.6 133.275) (size 0.5) (drill 0.3) (layers "F.Cu" "B.Cu") (net 4))
-  (via (at 123.9 133.275) (size 0.5) (drill 0.3) (layers "F.Cu" "B.Cu") (net 4))
   (via (at 118.3 133.275) (size 0.5) (drill 0.3) (layers "F.Cu" "B.Cu") (net 4))
   (via (at 132.5 133.275) (size 0.5) (drill 0.3) (layers "F.Cu" "B.Cu") (net 4))

Commit message: DAC8: 10uF bulk op VREF (ADR421-ontkoppeling per datasheet)
Cross-check tegen doc/data-sheets/AD5754BREZ data.md bevestigde de pinout
(3 bronnen) en dat de referentiepen 0,1uF + 10uF hoort te krijgen. C6 was
er al (0,1uF); C14 (10uF, oostrand tussen +12V-spine en C1) toegevoegd op
/VREF naast C6, U1.17, U2.17, U3.8. ERC 0, netcheck OK, DRC 0/0; PDF's +
fab herzien. README: BREZ heeft geen interne ref -> ADR421 verplicht.

Co-Authored-By: Claude Fable 5 <noreply@anthropic.com>
Parts:
- added C14: 10u, Capacitor_SMD:CP_Elec_4x5.3, F.Cu at (145.5, 141.0)
Routing:
- net /VREF: track 48.8 -> 66.7 mm, vias 4 -> 5
- net GND: track 4.05 -> 6.05 mm, vias 23 -> 24
