File: Images/schematics/musicbrain-adc8/musicbrain-adc8.kicad_sch (KiCad schematic)
At the start: 23 parts, among them J1 BUS, J2 CV IN, U1 AD7606BSTZ, U2 AMS1117-5.0

Commit message: ADC8 v1.1: haakse connectoren + volledige routing (DRC 0/0)
- bord van 80x44 naar 40x80 mm (H=80-standaard); J1 haaks onder,
  J2 haaks boven, gecentreerd boven het slot
- de v1.0-routing liep twee keer vast; de bovenplaat-layout lost het op:
  V1..V8 -> IN1..IN8 (volledige orde-omkering) via Manhattan-routing
  (F.Cu alleen verticalen, B.Cu 8 horizontale lanes op 0,8mm steek),
  westkolom-entries kruisingsvrij met 'diepste entry = oostelijkste
  verticaal', GND-verzamelrail voor de pads tussen de escapes
- ERC 0, netlijst pad-voor-pad geverifieerd, DRC 0/0 met zone-refill

Co-Authored-By: Claude Fable 5 <noreply@anthropic.com>
Parts:
- J1: footprint Connector_PinHeader_2.54mm:PinHeader_2x10_P2.54mm_Vertical -> Connector_PinHeader_2.54mm:PinHeader_2x10_P2.54mm_Horizontal
- J2: footprint Connector_PinHeader_2.54mm:PinHeader_1x10_P2.54mm_Vertical -> Connector_PinHeader_2.54mm:PinHeader_1x10_P2.54mm_Horizontal
Changed lines of the file:
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@@
     (property "Reference" "J1" (at 60 93.49 0) (effects (font (size 1.27 1.27))))
     (property "Value" "BUS" (at 60 126.51 0) (effects (font (size 1.27 1.27))))
-    (property "Footprint" "Connector_PinHeader_2.54mm:PinHeader_2x10_P2.54mm_Vertical" (at 60 110 0) (effects (font (size 1.27 1.27)) (hide yes)))
+    (property "Footprint" "Connector_PinHeader_2.54mm:PinHeader_2x10_P2.54mm_Horizontal" (at 60 110 0) (effects (font (size 1.27 1.27)) (hide yes)))
     (property "Datasheet" "" (at 60 110 0) (effects (font (size 1.27 1.27)) (hide yes)))
     (instances (project "musicbrain-adc8" (path "/f0000000-0000-4000-8000-000000000000" (reference "J1") (unit 1))))
@@
     (property "Reference" "J2" (at 215 106.03 0) (effects (font (size 1.27 1.27))))
     (property "Value" "CV IN" (at 215 136.51 0) (effects (font (size 1.27 1.27))))
-    (property "Footprint" "Connector_PinHeader_2.54mm:PinHeader_1x10_P2.54mm_Vertical" (at 215 120 0) (effects (font (size 1.27 1.27)) (hide yes)))
+    (property "Footprint" "Connector_PinHeader_2.54mm:PinHeader_1x10_P2.54mm_Horizontal" (at 215 120 0) (effects (font (size 1.27 1.27)) (hide yes)))
     (property "Datasheet" "" (at 215 120 0) (effects (font (size 1.27 1.27)) (hide yes)))
     (instances (project "musicbrain-adc8" (path "/f0000000-0000-4000-8000-000000000000" (reference "J2") (unit 1))))

Commit message: ADC8 v1.2: recht-toe-bedrading + firmware-remap (DRC 0/0 + fab)
V-omkering eruit: V_k nu recht naar paneeljack (9-k) via een ordebehoudende
F.Cu-waaier (geen B-lanes/vias meer). MbAdc8::read() spiegelt de AD7606-
stream zodat out[0..7] = paneeljack 1..8; jack-contract op J2 ongewijzigd.
ERC 0, netcheck OK, DRC 0/0, fab ververst (JLC-formaat) - bestelbaar.

Co-Authored-By: Claude Fable 5 <noreply@anthropic.com>
Parts:
- J1: footprint Connector_PinHeader_2.54mm:PinHeader_2x10_P2.54mm_Horizontal -> Connector_PinHeader_2.54mm:PinHeader_2x10_P2.54mm_Vertical
- J2: footprint Connector_PinHeader_2.54mm:PinHeader_1x10_P2.54mm_Horizontal -> Connector_PinHeader_2.54mm:PinHeader_1x10_P2.54mm_Vertical
Connections:
- net IN1: now also R8.2; no longer R1.2
- net IN2: now also R7.2; no longer R2.2
- net IN3: now also R6.2; no longer R3.2
- net IN4: now also R5.2; no longer R4.2
- net IN5: now also R4.2; no longer R5.2
- net IN6: now also R3.2; no longer R6.2
- net IN7: now also R2.2; no longer R7.2
- net IN8: now also R1.2; no longer R8.2
Changed lines of the file:
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@@
     (title "MusicBrain ADC8 - 8x CV input slot card")
     (date "2026-07-07")
-    (rev "1.0")
+    (rev "1.2")
     (company "MusicBrain project")
     (comment 1 "AD7606 16-bit 8-ch simultaneous SAR, +/-10V direct, serial mode")
@@
   )
   (wire (pts (xy 167.94 122.54) (xy 173.02 122.54)) (stroke (width 0) (type default)))
-  (label "IN1" (at 173.02 122.54 0) (effects (font (size 1.27 1.27)) (justify left bottom)))
+  (label "IN8" (at 173.02 122.54 0) (effects (font (size 1.27 1.27)) (justify left bottom)))
   (wire (pts (xy 157.78 125.08) (xy 162.86 125.08)) (stroke (width 0) (type default)))
   (symbol (lib_id "power:GND") (at 162.86 125.08 0)
@@
   )
   (wire (pts (xy 167.94 127.62) (xy 173.02 127.62)) (stroke (width 0) (type default)))
-  (label "IN2" (at 173.02 127.62 0) (effects (font (size 1.27 1.27)) (justify left bottom)))
+  (label "IN7" (at 173.02 127.62 0) (effects (font (size 1.27 1.27)) (justify left bottom)))
   (wire (pts (xy 157.78 130.16) (xy 162.86 130.16)) (stroke (width 0) (type default)))
   (symbol (lib_id "power:GND") (at 162.86 130.16 0)
@@
   )
   (wire (pts (xy 167.94 132.7) (xy 173.02 132.7)) (stroke (width 0) (type default)))
-  (label "IN3" (at 173.02 132.7 0) (effects (font (size 1.27 1.27)) (justify left bottom)))
+  (label "IN6" (at 173.02 132.7 0) (effects (font (size 1.27 1.27)) (justify left bottom)))
   (wire (pts (xy 157.78 135.24) (xy 162.86 135.24)) (stroke (width 0) (type default)))
   (symbol (lib_id "power:GND") (at 162.86 135.24 0)
@@
   )
   (wire (pts (xy 167.94 137.78) (xy 173.02 137.78)) (stroke (width 0) (type default)))
-  (label "IN4" (at 173.02 137.78 0) (effects (font (size 1.27 1.27)) (justify left bottom)))
+  (label "IN5" (at 173.02 137.78 0) (effects (font (size 1.27 1.27)) (justify left bottom)))
   (wire (pts (xy 157.78 140.32) (xy 162.86 140.32)) (stroke (width 0) (type default)))
   (symbol (lib_id "power:GND") (at 162.86 140.32 0)
@@
   )
   (wire (pts (xy 167.94 142.86) (xy 173.02 142.86)) (stroke (width 0) (type default)))
-  (label "IN5" (at 173.02 142.86 0) (effects (font (size 1.27 1.27)) (justify left bottom)))
+  (label "IN4" (at 173.02 142.86 0) (effects (font (size 1.27 1.27)) (justify left bottom)))
   (wire (pts (xy 157.78 145.4) (xy 162.86 145.4)) (stroke (width 0) (type default)))
   (symbol (lib_id "power:GND") (at 162.86 145.4 0)
@@
   )
   (wire (pts (xy 167.94 147.94) (xy 173.02 147.94)) (stroke (width 0) (type default)))
-  (label "IN6" (at 173.02 147.94 0) (effects (font (size 1.27 1.27)) (justify left bottom)))
+  (label "IN3" (at 173.02 147.94 0) (effects (font (size 1.27 1.27)) (justify left bottom)))
   (wire (pts (xy 157.78 150.48) (xy 162.86 150.48)) (stroke (width 0) (type default)))
   (symbol (lib_id "power:GND") (at 162.86 150.48 0)
@@
   )
   (wire (pts (xy 167.94 153.02) (xy 173.02 153.02)) (stroke (width 0) (type default)))
-  (label "IN7" (at 173.02 153.02 0) (effects (font (size 1.27 1.27)) (justify left bottom)))
+  (label "IN2" (at 173.02 153.02 0) (effects (font (size 1.27 1.27)) (justify left bottom)))
   (wire (pts (xy 157.78 155.56) (xy 162.86 155.56)) (stroke (width 0) (type default)))
   (symbol (lib_id "power:GND") (at 162.86 155.56 0)
@@
   )
   (wire (pts (xy 167.94 158.1) (xy 173.02 158.1)) (stroke (width 0) (type default)))
-  (label "IN8" (at 173.02 158.1 0) (effects (font (size 1.27 1.27)) (justify left bottom)))
+  (label "IN1" (at 173.02 158.1 0) (effects (font (size 1.27 1.27)) (justify left bottom)))
   (wire (pts (xy 157.78 160.64) (xy 162.86 160.64)) (stroke (width 0) (type default)))
   (symbol (lib_id "power:GND") (at 162.86 160.64 0)
@@
     (property "Reference" "J1" (at 60 93.49 0) (effects (font (size 1.27 1.27))))
     (property "Value" "BUS" (at 60 126.51 0) (effects (font (size 1.27 1.27))))
-    (property "Footprint" "Connector_PinHeader_2.54mm:PinHeader_2x10_P2.54mm_Horizontal" (at 60 110 0) (effects (font (size 1.27 1.27)) (hide yes)))
+    (property "Footprint" "Connector_PinHeader_2.54mm:PinHeader_2x10_P2.54mm_Vertical" (at 60 110 0) (effects (font (size 1.27 1.27)) (hide yes)))
     (property "Datasheet" "" (at 60 110 0) (effects (font (size 1.27 1.27)) (hide yes)))
     (instances (project "musicbrain-adc8" (path "/f0000000-0000-4000-8000-000000000000" (reference "J1") (unit 1))))
@@
     (property "Reference" "J2" (at 215 106.03 0) (effects (font (size 1.27 1.27))))
     (property "Value" "CV IN" (at 215 136.51 0) (effects (font (size 1.27 1.27))))
-    (property "Footprint" "Connector_PinHeader_2.54mm:PinHeader_1x10_P2.54mm_Horizontal" (at 215 120 0) (effects (font (size 1.27 1.27)) (hide yes)))
+    (property "Footprint" "Connector_PinHeader_2.54mm:PinHeader_1x10_P2.54mm_Vertical" (at 215 120 0) (effects (font (size 1.27 1.27)) (hide yes)))
     (property "Datasheet" "" (at 215 120 0) (effects (font (size 1.27 1.27)) (hide yes)))
     (instances (project "musicbrain-adc8" (path "/f0000000-0000-4000-8000-000000000000" (reference "J2") (unit 1))))
