File: hardware/schematics/musicbrain-pot8front/musicbrain-pot8front.kicad_pcb (KiCad board)
At the start: 2 copper layers, 20 x 110 mm, 9 parts, among them J1 SOCKET-BACK

Commit message: jack8/jack4 v1.2 + pot8front v1.1: koppel-standaard + 3D-socket-fix
- Front-koppeling gestandaardiseerd: 1x10-socket op x=116,5 (16,5 van west-
  rand), pin 1 op y=143,57 - identiek op jack8, jack4 en pot8front
- B-zijde-sockets nu in KiCads canonieke geflipte vorm (rot 180, lokale y
  genegeerd): koper ongewijzigd, maar het 3D-model staat nu OP de gatenrij
  i.p.v. ernaast gespiegeld
- PCB-papier naar A3 (borden vielen van A4-landscape af), silk-URL naar
  bordmidden (viel over de bordrand door center-justify)
- make_fab.sh: bordenlijst actueel (deprecated eruit, fronts erin),
  selectie-argument + gerber-zip-stap toegevoegd
- ERC/netcheck/DRC 0/0 op alle drie; fab + PDF's ververst

Co-Authored-By: Claude Fable 5 <noreply@anthropic.com>
Parts:
- turned J1 to 180 degrees
Other:
- board text added: "musicbrain.nl/hw/pot8front rev 1.1"
- board text removed: "musicbrain.nl/hw/pot8front rev 1.0"
Changed lines of the file:
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@@
   (generator_version "8.0")
   (general (thickness 1.6) (legacy_teardrops no))
-  (paper "A4")
+  (paper "A3")
   (title_block
     (title "MusicBrain POT8-FRONT")
     (date "2026-07-11")
-    (rev "1.0")
+    (rev "1.1")
     (company "MusicBrain project")
   )
@@
   (footprint "MusicBrain:Socket_1x10_backside"
     (layer "B.Cu")
-    (at 116.5 143.57)
+    (at 116.5 143.57 180)
     (descr "1x10 female socket op de achterzijde; opening omlaag naar riser/kaart")
-    (property "Reference" "J1" (at 2.8 -2.2 0) (layer "B.SilkS")
+    (property "Reference" "J1" (at -2.8 2.2 0) (layer "B.SilkS")
       (effects (font (size 1 1) (thickness 0.15)) (justify mirror)))
-    (property "Value" "SOCKET-BACK" (at 0 25.9 0) (layer "B.Fab")
+    (property "Value" "SOCKET-BACK" (at 0 -25.9 0) (layer "B.Fab")
       (effects (font (size 1 1) (thickness 0.15)) (justify mirror)))
     (attr through_hole)
-    (fp_rect (start -1.6 -1.6) (end 1.6 24.46)
+    (fp_rect (start -1.6 -24.46) (end 1.6 1.6)
       (stroke (width 0.12) (type solid)) (fill no) (layer "B.SilkS"))
-    (fp_rect (start -1.8 -1.8) (end 1.8 24.66)
+    (fp_rect (start -1.8 -24.66) (end 1.8 1.8)
       (stroke (width 0.05) (type solid)) (fill no) (layer "B.CrtYd"))
-    (pad "1" thru_hole rect (at 0 0) (size 1.7 1.7) (drill 1.0) (layers "*.Cu" "*.Mask") (net 1 "GND"))
-    (pad "2" thru_hole oval (at 0 2.54) (size 1.7 1.7) (drill 1.0) (layers "*.Cu" "*.Mask") (net 3 "/W1"))
-    (pad "3" thru_hole oval (at 0 5.08) (size 1.7 1.7) (drill 1.0) (layers "*.Cu" "*.Mask") (net 4 "/W2"))
-    (pad "4" thru_hole oval (at 0 7.62) (size 1.7 1.7) (drill 1.0) (layers "*.Cu" "*.Mask") (net 5 "/W3"))
-    (pad "5" thru_hole oval (at 0 10.16) (size 1.7 1.7) (drill 1.0) (layers "*.Cu" "*.Mask") (net 6 "/W4"))
-    (pad "6" thru_hole oval (at 0 12.7) (size 1.7 1.7) (drill 1.0) (layers "*.Cu" "*.Mask") (net 7 "/W5"))
-    (pad "7" thru_hole oval (at 0 15.24) (size 1.7 1.7) (drill 1.0) (layers "*.Cu" "*.Mask") (net 8 "/W6"))
-    (pad "8" thru_hole oval (at 0 17.78) (size 1.7 1.7) (drill 1.0) (layers "*.Cu" "*.Mask") (net 9 "/W7"))
-    (pad "9" thru_hole oval (at 0 20.32) (size 1.7 1.7) (drill 1.0) (layers "*.Cu" "*.Mask") (net 10 "/W8"))
-    (pad "10" thru_hole oval (at 0 22.86) (size 1.7 1.7) (drill 1.0) (layers "*.Cu" "*.Mask") (net 2 "+3V3"))
+    (pad "1" thru_hole rect (at 0 -0 180) (size 1.7 1.7) (drill 1.0) (layers "*.Cu" "*.Mask") (net 1 "GND"))
+    (pad "2" thru_hole oval (at 0 -2.54 180) (size 1.7 1.7) (drill 1.0) (layers "*.Cu" "*.Mask") (net 3 "/W1"))
+    (pad "3" thru_hole oval (at 0 -5.08 180) (size 1.7 1.7) (drill 1.0) (layers "*.Cu" "*.Mask") (net 4 "/W2"))
+    (pad "4" thru_hole oval (at 0 -7.62 180) (size 1.7 1.7) (drill 1.0) (layers "*.Cu" "*.Mask") (net 5 "/W3"))
+    (pad "5" thru_hole oval (at 0 -10.16 180) (size 1.7 1.7) (drill 1.0) (layers "*.Cu" "*.Mask") (net 6 "/W4"))
+    (pad "6" thru_hole oval (at 0 -12.7 180) (size 1.7 1.7) (drill 1.0) (layers "*.Cu" "*.Mask") (net 7 "/W5"))
+    (pad "7" thru_hole oval (at 0 -15.24 180) (size 1.7 1.7) (drill 1.0) (layers "*.Cu" "*.Mask") (net 8 "/W6"))
+    (pad "8" thru_hole oval (at 0 -17.78 180) (size 1.7 1.7) (drill 1.0) (layers "*.Cu" "*.Mask") (net 9 "/W7"))
+    (pad "9" thru_hole oval (at 0 -20.32 180) (size 1.7 1.7) (drill 1.0) (layers "*.Cu" "*.Mask") (net 10 "/W8"))
+    (pad "10" thru_hole oval (at 0 -22.86 180) (size 1.7 1.7) (drill 1.0) (layers "*.Cu" "*.Mask") (net 2 "+3V3"))
     (model "${KICAD10_3DMODEL_DIR}/Connector_PinSocket_2.54mm.3dshapes/PinSocket_1x10_P2.54mm_Vertical.step"
       (offset (xyz 0 0 0)) (scale (xyz 1 1 1)) (rotate (xyz 0 0 0)))
@@
     (stroke (width 0.1) (type default)) (fill none)
     (layer "Edge.Cuts"))
-  (gr_text "musicbrain.nl/hw/pot8front rev 1.0" (at 101.3 206 90) (layer "F.SilkS")
+  (gr_text "musicbrain.nl/hw/pot8front rev 1.1" (at 101.3 155 90) (layer "F.SilkS")
     (effects (font (size 1 1) (thickness 0.15))))
   (gr_text "as-hartlijn 8.0" (at 108 101.2 0) (layer "F.Fab")
