File: hardware/schematics/gswitch-brain/gswitch-brain.kicad_pcb (KiCad board)
At the start: 2 copper layers, 100 x 70 mm, 69 parts, among them J1 DC-12V, J10 RJ45-S, J11 RJ45-S, J2 USB-C, J3 SDS-50J, J4 SDS-50J, J5 OLED-I2C, J6 KNOPPEN, J7 ENCODER, J8 SPARE, J9 DEBUG, Q1 AO3401, SW1 RESET, SW2 BOOT, U1 ESP32-S3-WROOM-1U-N8R2, U2 74HCT541, U3 74HCT14, U4 H11L1, U5 AMS1117-3.3, U6 TPS563201

Commit message: gswitch-brain: silk-labels op Marks indeling + grafisch aansluitoverzicht
Silk: titel en 12V-center-negatief-regel tussen de RJ45s, spec-URL 90
graden langs de oostrand (de oude onderrand-regel verdween onder J11/H4);
generator ondersteunt nu meerdere silk-teksten (b.silk_texts).

Nieuw: gswitch_overzicht.py - kicad-cli svg-export + callouts in
bordcoordinaten -> gswitch-brain-overzicht.svg, gelinkt in de README.

Co-Authored-By: Claude Fable 5 <noreply@anthropic.com>
Other:
- board text added: "12V center-negatief"
- board text added: "GSWITCH BRAIN rev 0.1"
- board text added: "doc/guitar-switcher-spec.md"
- board text removed: "GSWITCH BRAIN rev 0.1 - 12V center-negatief - doc/guitar-switcher-spec.md"
Changed lines of the file:
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@@
     (stroke (width 0.1) (type default)) (fill none)
     (layer "Edge.Cuts"))
-  (gr_text "GSWITCH BRAIN rev 0.1 - 12V center-negatief - doc/guitar-switcher-spec.md" (at 150 167.3 0) (layer "F.SilkS")
+  (gr_text "GSWITCH BRAIN rev 0.1" (at 146 153.9 0) (layer "F.SilkS")
+    (effects (font (size 1 1) (thickness 0.15))))
+  (gr_text "12V center-negatief" (at 146 157 0) (layer "F.SilkS")
+    (effects (font (size 1 1) (thickness 0.15))))
+  (gr_text "doc/guitar-switcher-spec.md" (at 184.6 156.5 90) (layer "F.SilkS")
     (effects (font (size 1 1) (thickness 0.15))))
   (zone (net 4) (net_name "GND") (layer "F.Cu")
