File: hardware/schematics/musicbrain-busboard-v2/musicbrain-busboard-v2.kicad_sch (KiCad schematic)
At the start: 89 parts, among them J1 SLOT 1, J10 EXP, J11 DISPLAY, J12 QWIIC, J13 MIDI IN1, J14 MIDI IN2, J15 MIDI OUT, J16 CAN, J17 AUDIO/CODEC, J18 TUNE, J19 DLG1 (Serial3), J2 SLOT 2, J20 DLG2 (Serial4), J21 EXPANSION, J3 SLOT 3, J4 SLOT 4, J5 SLOT 5, J6 SLOT 6, J7 HUB 1, J8 HUB 2, J9 PWR IN, U1 Teensy 4.1, U10 H11L1, U11 74LVC1G17, U12 SN65HVD230, U13 74LVC1G17, U2 R-78E5.0-0.5, U3 AMS1117-3.3, U4 74HC154, U5 74HC165, U6 74HC165, U7 74LVC1G125, U8 74LVC245, U9 H11L1

Commit message: jlc_fix: haakse slotkaart-headers + JP1/knopjes; AD5754-rotatie; fab herzien
Library uitgebreid en fab van alle borden opnieuw gegenereerd met de nieuwe
inzichten uit de JLCPCB-preview + de offline parts-catalogus:
- ROT_FIX: AD5754 (HTSSOP-24) +270 (geverifieerd); SOIC-16 geldt cross-chip
  (74HC165/74HCT595/MCP3208), SOIC-8 (SN65HVD230/ADR421), LQFP-64/QFN-28 = raw.
- Haakse slotkaart-headers: J1 BUS -> C19190505, J2 CV/gates -> C2687688
  (dac8/gate8/gatein8; adc8 staat nog op Vertical = board-fix, zie MODULES).
- adc8 JP1 RANGE -> C49257 (recht 1x3; comment-specifiek, busboard-MIDI blijft
  leeg). enc5front-knopjes SW6/SW7 -> C110153 (6x6mm THT).

WERKWIJZE: FTS-zoekvocabulaire (AND/exact, geen streepjes/2.54mm-token; male =
"Pin Header 2x10P", haaks = "Right Angle"). busboard J11-label -> "connector
to DISPLAY".
Parts:
- J11: value DISPLAY -> connector to DISPLAY
Changed lines of the file:
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@@
     (unit 1) (exclude_from_sim no) (in_bom yes) (on_board yes) (dnp no)
     (property "Reference" "J11" (at 225 264 0) (effects (font (size 1.27 1.27))))
-    (property "Value" "DISPLAY" (at 225 292 0) (effects (font (size 1.27 1.27))))
+    (property "Value" "connector to DISPLAY" (at 225 292 0) (effects (font (size 1.27 1.27))))
     (property "Footprint" "Connector_PinHeader_2.54mm:PinHeader_1x09_P2.54mm_Vertical" (at 225 278 0) (effects (font (size 1.27 1.27)) (hide yes)))
     (property "Datasheet" "" (at 225 278 0) (effects (font (size 1.27 1.27)) (hide yes)))
