File: hardware/schematics/musicbrain-adc8/musicbrain-adc8.kicad_sch (KiCad schematic)
At the start: 23 parts, among them J1 BUS, J2 CV IN, U1 AD7606BSTZ, U2 AMS1117-5.0

Commit message: adc8: schema-footprint J1/J2 -> Horizontal (was uit sync met PCB)
De adc8-PCB gebruikte al haakse headers (PinHeader_2x10/1x10_Horizontal), maar
het schema-footprintveld (en de generators) stonden nog op _Vertical. Daardoor
zei de BOM "Vertical" en matchte de haakse header-library er niet op. PCB/koper/
routing waren correct; alleen de metadata is rechtgetrokken (schema + gen_adc_
sch/pcb). BOM pakt nu J1->C19190505, J2->C2687688.

Co-Authored-By: Claude Opus 4.8 <noreply@anthropic.com>
Parts:
- J1: footprint Connector_PinHeader_2.54mm:PinHeader_2x10_P2.54mm_Vertical -> Connector_PinHeader_2.54mm:PinHeader_2x10_P2.54mm_Horizontal
- J2: footprint Connector_PinHeader_2.54mm:PinHeader_1x10_P2.54mm_Vertical -> Connector_PinHeader_2.54mm:PinHeader_1x10_P2.54mm_Horizontal
Changed lines of the file:
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@@
     (property "Reference" "J1" (at 60 93.49 0) (effects (font (size 1.27 1.27))))
     (property "Value" "BUS" (at 60 126.51 0) (effects (font (size 1.27 1.27))))
-    (property "Footprint" "Connector_PinHeader_2.54mm:PinHeader_2x10_P2.54mm_Vertical" (at 60 110 0) (effects (font (size 1.27 1.27)) (hide yes)))
+    (property "Footprint" "Connector_PinHeader_2.54mm:PinHeader_2x10_P2.54mm_Horizontal" (at 60 110 0) (effects (font (size 1.27 1.27)) (hide yes)))
     (property "Datasheet" "" (at 60 110 0) (effects (font (size 1.27 1.27)) (hide yes)))
     (instances (project "musicbrain-adc8" (path "/f0000000-0000-4000-8000-000000000000" (reference "J1") (unit 1))))
@@
     (property "Reference" "J2" (at 215 106.03 0) (effects (font (size 1.27 1.27))))
     (property "Value" "CV IN" (at 215 136.51 0) (effects (font (size 1.27 1.27))))
-    (property "Footprint" "Connector_PinHeader_2.54mm:PinHeader_1x10_P2.54mm_Vertical" (at 215 120 0) (effects (font (size 1.27 1.27)) (hide yes)))
+    (property "Footprint" "Connector_PinHeader_2.54mm:PinHeader_1x10_P2.54mm_Horizontal" (at 215 120 0) (effects (font (size 1.27 1.27)) (hide yes)))
     (property "Datasheet" "" (at 215 120 0) (effects (font (size 1.27 1.27)) (hide yes)))
     (instances (project "musicbrain-adc8" (path "/f0000000-0000-4000-8000-000000000000" (reference "J2") (unit 1))))

Commit message: adc8 gen 2: 80x45, slot 2x12, RESET lokaal, GND-binnenring
- kaart 50x80 -> 80x45; J1 2x10 -> 2x12 via bus.j1_map; pin 19 = /SPARE1
  = busbrede CONVST; J2 gecentreerd
- RESET van buslijn (SPARE2, vervallen in gen 2) naar lokale RC-power-up:
  C15 100n vanaf +3V3 + R9 100k pulldown (tau 10 ms)
- U1 rot 0: V-ingangen noord naar de IN-kolommen; v1.2-mapping (jack j =
  V(9-j), remap in MbAdc8) blijft
- GND-binnenring onder de LQFP: zone-vulling bereikt 0,5mm-pads nooit
  (0,6 mm kanaal nodig); straps + ring + 2 via's, zoals gen-1 met de hand
- prep_dsn --route-gnd: GND blijft routeerbaar net (alleen planes eruit),
  zodat freerouting de vaste GND-wiring ziet en zelf GND afmaakt
- gen_adc_pcb.py (cardlib) vervangt gen_adc_pcb_v11.py + oude gen_adc_pcb.py
- ERC 0, netcheck OK, DRC 0/0

Co-Authored-By: Claude Fable 5 <noreply@anthropic.com>
Parts:
- removed R2, R7: 1k, Resistor_SMD:R_0805_2012Metric, symbol Device:R
- removed R9: 100k, Resistor_SMD:R_0805_2012Metric, symbol Device:R
- added C15, C4: 100n, Capacitor_SMD:C_0805_2012Metric, symbol Device:C
- added J1: BUS (slot, 2x12), Connector_PinHeader_2.54mm:PinHeader_2x12_P2.54mm_Horizontal, symbol Custom:Conn_02x12
- added R3: 1k, Resistor_SMD:R_0805_2012Metric, symbol Device:R
- R7: renamed from J1; value BUS -> 1k; footprint Connector_PinHeader_2.54mm:PinHeader_2x10_P2.54mm_Horizontal -> Resistor_SMD:R_0805_2012Metric; symbol Custom:Conn_02x10 -> Device:R
- R9: renamed from C4; value 100n -> 100k; footprint Capacitor_SMD:C_0805_2012Metric -> Resistor_SMD:R_0805_2012Metric; symbol Device:C -> Device:R
- renumbered R3 to R2
Connections:
- net +12V: now also J1.2 (Pin_2); no longer R7.2 (Pin_2)
- net +3V3: now also C15.1, J1.6 (Pin_6); no longer R7.6 (Pin_6)
- net +5V: now also C4.1; no longer R9.1
- net CONVST: now also J1.19 (Pin_19); no longer R7.19 (Pin_19)
- net CS: now also J1.13 (Pin_13); no longer R7.13 (Pin_13)
- net GND: now also C4.2, J1.1 (Pin_1), J1.10 (Pin_10), J1.12 (Pin_12), J1.14 (Pin_14), J1.20 (Pin_20), J1.3 (Pin_3), J1.5 (Pin_5), J1.8 (Pin_8); no longer R7.1 (Pin_1), R7.10 (Pin_10), R7.12 (Pin_12), R7.14 (Pin_14), R7.3 (Pin_3), R7.5 (Pin_5), R7.8 (Pin_8)
- net IN2: now also R7.2
- net IN6: now also R3.2; no longer R2.2
- net IN7: now also R2.2
- net IRQ: now also J1.16 (Pin_16); no longer R7.16 (Pin_16)
- net MISO: now also J1.11 (Pin_11); no longer R7.11 (Pin_11)
- net RESET: now also R9.1, C15.2; no longer R7.20 (Pin_20)
- net SCLK: now also J1.7 (Pin_7); no longer R7.7 (Pin_7)
- net REGCAP1: now reaches C6.1, U1.36 (REGCAP1)
- net REGCAP2: now reaches C7.1, U1.39 (REGCAP2)
- net REF: now reaches C8.1, U1.42 (REFIN/REFOUT)
- net REFCAP: now reaches C9.1, U1.44 (REFCAPA), U1.45 (REFCAPB)
- net V1: now reaches R1.1, U1.49 (V1)
- net V2: now reaches U1.51 (V2)
- net V2: now also R2.1
- net V3: now reaches U1.53 (V3)
- net V3: now also R3.1; no longer R2.1
- net V4: now reaches R4.1, U1.55 (V4)
- net V5: now reaches R5.1, U1.57 (V5)
- net V6: now reaches R6.1, U1.59 (V6)
- net V7: now reaches U1.61 (V7)
- net V7: now also R7.1
- net V8: now reaches R8.1, U1.63 (V8)
- no-connect marks 7 -> 11
Other:
- note added: "AD7606: 16-bit, 8-ch simultaneous, +/-10V or +/-5V direct in (1 Mohm, clamps) Serial mode: PAR/SER=high, DB0-6/DB9-15=GND, DOUTA=MISO, DOUTB=nc Internal 2.5V ref (REF_SELECT=high); REGCAP 2x1u, REFCAP 10u, REFIN 10u CONVST=SPARE1/pin19 (bus-wide sample strobe); RESET=lokale RC-power-up (C15/R9) BUSY -> IRQ (falling edge = data ready); RANGE via JP1: +3V3=+/-10V, GND=+/-5V AVCC=5V local (AMS1117-5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"
- note removed: "AD7606: 16-bit, 8-ch simultaneous, +/-10V or +/-5V direct in (1 Mohm, clamps) Serial mode: PAR/SER=high, DB0-6/DB9-15=GND, DOUTA=MISO, DOUTB=nc Internal 2.5V ref (REF_SELECT=high); REGCAP 2x1u, REFCAP 10u, REFIN 10u CONVST=SPARE1 (bus-wide sample strobe), RESET=SPARE2 (+100k pulldown) BUSY -> IRQ (falling edge = data ready); RANGE via JP1: +3V3=+/-10V, GND=+/-5V AVCC=5V local (AMS1117-5.0), VDRIV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"
- moved on the sheet: R2
