File: hardware/schematics/musicbrain-busboard/musicbrain-busboard.kicad_pcb (KiCad board)
At the start: 2 copper layers, 203.2 x 128.5 mm, 102 parts, among them J1 SLOT 1, J10 EXP, J11 DISPLAY, J12 QWIIC, J13 MIDI IN1, J14 MIDI IN2, J15 MIDI OUT, J16 CAN, J17 AUDIO/CODEC, J18 TUNE, J19 DLG1, J2 SLOT 2, J20 DLG2, J21 EXPANSION, J22 MIDI OUT2, J23 USB HOST, J24 AUDIOHUB, J3 SLOT 3, J4 SLOT 4, J5 SLOT 5, J6 SLOT 6, J7 HUB 1, J8 HUB 2, J9 PWR IN, U1 Teensy 4.1, U10 H11L1, U11 74LVC1G17, U12 SN65HVD230, U13 74LVC1G17, U14 74LVC1G17, U2 R-78E5.0-1.0, U3 AMS1117-3.3, U4 74HC154, U5 74HC165, U6 74HC165, U7 74LVC1G125, U8 74LVC245, U9 H11L1

Commit message: busboard v3 AF: ERC 0, netcheck OK, DRC 0/0 (gen 2, rev 3.0)
Koper: freerouting best-of-4 (alle runs compleet na twee placement-
verbeteringen) + GND-hechtcyclus + 2 handmatige brugvia's.

Placement-lessen onderweg:
- U4 (74HC154) uit de Teensy/slot-1-gang naar de noordstrook: het
  gecentreerde slotveld maakte die gang 6 mm smaller dan v2 en
  /MOSI//CS3//BCLK bleven er consequent in steken; met de decoder
  noord (CS-waaier zuid naar de slots, oost naar J21) route alles
- CAN-cluster (U12 c.s.) naar het open zuidoosten: de GND-pad zat
  bij de MIDI-cluster ingesloten zonder via-plek
- gnd_bridge zoekt alleen B-hoofdvlak-onder-F-fragment; de twee
  spiegelgevallen (grote losse B-stroken onder de laanbundel) met een
  eigen scan gedicht: brugvia's (73.83,95) en (72.89,87.54)
- MCP-les: na regeneratie eerst het project herladen, anders
  exporteert export_dsn het gecachte oude bord

Co-Authored-By: Claude Fable 5 <noreply@anthropic.com>
Parts:
- moved R13 60.2 mm to (150.0, 118.0)
- moved JP1 58.0 mm to (157.5, 117.5)
- moved U12 58.0 mm to (150.0, 112.0)
- moved C13 55.4 mm to (143.0, 112.0), turned to 0 degrees
- moved R12 55.1 mm to (158.0, 112.0)
- moved C10 42.1 mm to (60.0, 27.0), turned to 0 degrees
- moved U4 29.7 mm to (70.0, 32.0), turned to 90 degrees
Routing:
- net +3V3: track 0.00 -> 753.3 mm, vias 0 -> 5
- net +12V: track 0.00 -> 478.8 mm, vias 0 -> 2
- net -12V: track 0.00 -> 421.7 mm, vias 0 -> 2
- net /MISO: track 0.00 -> 359.0 mm, vias 0 -> 2
- net /SCLK: track 0.00 -> 358.5 mm, vias 0 -> 4
- net /SDA: track 0.00 -> 295.1 mm, vias 0 -> 4
- net /SCL: track 0.00 -> 294.7 mm, vias 0 -> 4
- net +5V: track 0.00 -> 284.5 mm, vias 0 -> 4
- net /LRCLK: track 0.00 -> 268.6 mm, vias 0 -> 3
- net /MOSI: track 0.00 -> 251.5 mm, vias 0 -> 3
- net /BCLK: track 0.00 -> 234.5 mm, vias 0 -> 4
- net /MCLK: track 0.00 -> 228.1 mm, vias 0 -> 4
- net /CHAIN: track 0.00 -> 219.6 mm, vias 0 -> 2
- net /LDAC: track 0.00 -> 218.5 mm, vias 0 -> 1
- net /IRQSTAT: track 0.00 -> 209.1 mm, vias 0 -> 4
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
Commit message: busboard v3: J24 naar de oostrand (mechanica-vangst Mark) + GND geroute
- J24 audiohub van midden-zuid naar de oostrand tussen de hubs: de
  kaarten beslaan y 34..114 op de slotvlakken - een kabel midden op het
  bord kan nergens heen; DRC ziet zoiets niet
- herroute met prep_dsn --route-gnd: de router schampte netloze
  GND-pads (geen clearance zonder net) en de zone-eilanden bleven
  terugkomen; met GND als net is het in een run schoon en zijn de
  hechtvia-rondes overbodig (vlakken = bonuskoper)
- SES-apply neemt GND nu wel mee uit de SES
- ERC 0, netcheck OK, DRC 0/0

Co-Authored-By: Claude Fable 5 <noreply@anthropic.com>
Parts:
- moved J24 73.8 mm to (182.0, 72.0), turned to 0 degrees
Routing:
- net GND: track 0.00 -> 1599.1 mm, vias 41 -> 46
- net /I2SD3: track 29.8 -> 112.5 mm, vias 0 -> 2
- net /I2SD2: track 42.8 -> 118.6 mm, vias 0 -> 1
- net /I2SD1: track 65.2 -> 129.7 mm, vias 0 -> 3
- net /I2SD4: track 12.4 -> 71.1 mm
- net /MOSI: track 251.5 -> 298.3 mm
- net /MISO: track 359.0 -> 315.0 mm, vias 2 -> 5
- net /CS3: track 73.4 -> 108.2 mm
- net +3V3: track 753.3 -> 719.0 mm, vias 5 -> 4
- net /CS4: track 86.2 -> 116.1 mm
- net +12V: track 478.8 -> 506.8 mm, vias 2 -> 4
- net /TUNE_T: track 45.3 -> 66.8 mm
- net /I2SD6: track 43.5 -> 23.5 mm
- net /XLDAC0: track 15.4 -> 34.1 mm
- net /IRQSTAT: track 209.1 -> 192.1 mm, vias 4 -> 6
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
Commit message: busboard rev 3.1: J25 Axon-voedingsheader (+5V/GND naast J19)
Pin 1 landt op het +5V-spoor van de SES-bundel, pin 2 GND-stub naar de
GND-verticaal (x=70); geen herroute — ERC 0, netcheck OK, DRC 0/0.
Fab-pakket + assets + pinout J25 + README/MODULES bijgewerkt.

Co-Authored-By: Claude Fable 5 <noreply@anthropic.com>
Parts:
- added H6: M3, MountingHole:MountingHole_3.2mm_M3, F.Cu at (213.0, 133.5)
- C14: renamed from J23; value USB HOST -> 100n; footprint Connector_PinHeader_2.54mm:PinHeader_2x05_P2.54mm_Vertical -> Capacitor_SMD:C_0805_2012Metric
- C18: renamed from C10; value 100n -> 220p
- C19: renamed from R21; value 100k -> 100n; footprint Resistor_SMD:R_0805_2012Metric -> Capacitor_SMD:C_0805_2012Metric
- C9: renamed from R33; value 10k -> 220p; footprint Resistor_SMD:R_0805_2012Metric -> Capacitor_SMD:C_0805_2012Metric
- D2: renamed from R8; value 1k -> 1N4148WS; footprint Resistor_SMD:R_0805_2012Metric -> Diode_SMD:D_SOD-323
- D3: renamed from R14; value 100k -> BAT54S; footprint Resistor_SMD:R_0805_2012Metric -> Package_TO_SOT_SMD:SOT-23
- J11: renamed from J17; value AUDIO/CODEC -> DISPLAY; footprint Connector_PinHeader_2.54mm:PinHeader_2x07_P2.54mm_Vertical -> Connector_PinHeader_2.54mm:PinHeader_1x09_P2.54mm_Vertical
- J12: renamed from J11; value DISPLAY -> QWIIC; footprint Connector_PinHeader_2.54mm:PinHeader_1x09_P2.54mm_Vertical -> Connector_PinHeader_2.54mm:PinHeader_1x04_P2.54mm_Vertical
- J13: renamed from J14; value MIDI IN2 -> MIDI IN1
- J14: renamed from J15; value MIDI OUT -> MIDI IN2
- J15: renamed from J22; value MIDI OUT2 -> MIDI OUT
- J16: renamed from J12; value QWIIC -> CAN
- J17: renamed from J18; value TUNE -> AUDIO/CODEC; footprint Connector_PinHeader_2.54mm:PinHeader_1x02_P2.54mm_Vertical -> Connector_PinHeader_2.54mm:PinHeader_2x07_P2.54mm_Vertical
- J18: renamed from U13; value 74LVC1G17 -> TUNE; footprint Package_TO_SOT_SMD:SOT-23-5 -> Connector_PinHeader_2.54mm:PinHeader_1x02_P2.54mm_Vertical
- J20: renamed from J13; value MIDI IN1 -> DLG2; footprint Connector_PinHeader_2.54mm:PinHeader_1x03_P2.54mm_Vertical -> Connector_PinHeader_2.54mm:PinHeader_1x04_P2.54mm_Vertical
- J21: renamed from J24; value AUDIOHUB -> EXPANSION; footprint Connector_PinHeader_2.54mm:PinHeader_2x07_P2.54mm_Vertical -> Connector_IDC:IDC-Header_2x13_P2.54mm_Vertical
- J22: renamed from J16; value CAN -> MIDI OUT2; footprint Connector_PinHeader_2.54mm:PinHeader_1x04_P2.54mm_Vertical -> Connector_PinHeader_2.54mm:PinHeader_1x03_P2.54mm_Vertical
- J23: renamed from U4; value 74HC154 -> USB HOST; footprint Package_SO:SOIC-24W_7.5x15.4mm_P1.27mm -> Connector_PinHeader_2.54mm:PinHeader_2x05_P2.54mm_Vertical
- J24: renamed from U12; value SN65HVD230 -> AUDIOHUB; footprint Package_SO:SOIC-8_3.9x4.9mm_P1.27mm -> Connector_PinHeader_2.54mm:PinHeader_2x07_P2.54mm_Vertical
- J25: renamed from J20; value DLG2 -> AXON +5V; footprint Connector_PinHeader_2.54mm:PinHeader_1x04_P2.54mm_Vertical -> Connector_PinHeader_2.54mm:PinHeader_1x02_P2.54mm_Vertical
- JP1: renamed from H1; value M3 -> TERM; footprint MountingHole:MountingHole_3.2mm_M3 -> Jumper:SolderJumper-2_P1.3mm_Open_TrianglePad1.0x1.5mm
- R10: renamed from R11; value 33R -> 10R
- R11: renamed from R34; value 10R -> 33R
- R12: renamed from JP1; value TERM -> 120R; footprint Jumper:SolderJumper-2_P1.3mm_Open_TrianglePad1.0x1.5mm -> Resistor_SMD:R_0805_2012Metric
- R13: renamed from R12; value 120R -> 10k
- R15: renamed from C14; value 100n -> 100k; footprint Capacitor_SMD:C_0805_2012Metric -> Resistor_SMD:R_0805_2012Metric
- R20: renamed from R6; value 220R -> 33R
- R32: renamed from R16; value 33R -> 100k
- R33: renamed from C18; value 220p -> 10k; footprint Capacitor_SMD:C_0805_2012Metric -> Resistor_SMD:R_0805_2012Metric
- R34: renamed from R35; value 33R -> 10R
- R35: renamed from R13; value 10k -> 33R
- R5: renamed from C9; value 220p -> 10k; footprint Capacitor_SMD:C_0805_2012Metric -> Resistor_SMD:R_0805_2012Metric
- R7: renamed from D1; value 1N4148WS -> 220R; footprint Diode_SMD:D_SOD-323 -> Resistor_SMD:R_0805_2012Metric
- R9: renamed from R10; value 10R -> 1k
- U10: renamed from U11; value 74LVC1G17 -> H11L1; footprint Package_TO_SOT_SMD:SOT-23-5 -> Package_DIP:DIP-6_W7.62mm
- U12: renamed from U9; value H11L1 -> SN65HVD230; footprint Package_DIP:DIP-6_W7.62mm -> Package_SO:SOIC-8_3.9x4.9mm_P1.27mm
- U13: renamed from D3; value BAT54S -> 74LVC1G17; footprint Package_TO_SOT_SMD:SOT-23 -> Package_TO_SOT_SMD:SOT-23-5
- U14: renamed from R5; value 10k -> 74LVC1G17; footprint Resistor_SMD:R_0805_2012Metric -> Package_TO_SOT_SMD:SOT-23-5
- U4: renamed from U5; value 74HC165 -> 74HC154; footprint Package_SO:SOIC-16_3.9x9.9mm_P1.27mm -> Package_SO:SOIC-24W_7.5x15.4mm_P1.27mm
- U6: renamed from U7; value 74LVC1G125 -> 74HC165; footprint Package_TO_SOT_SMD:SOT-23-5 -> Package_SO:SOIC-16_3.9x9.9mm_P1.27mm
- U7: renamed from U8; value 74LVC245 -> 74LVC1G125; footprint Package_SO:SOIC-20W_7.5x12.8mm_P1.27mm -> Package_TO_SOT_SMD:SOT-23-5
- U8: renamed from J21; value EXPANSION -> 74LVC245; footprint Connector_IDC:IDC-Header_2x13_P2.54mm_Vertical -> Package_SO:SOIC-20W_7.5x12.8mm_P1.27mm
- moved H3 214.9 mm to (213.0, 15.0)
- moved J12 201.1 mm to (198.0, 135.0)
- moved JP1 173.3 mm to (157.5, 117.5)
- moved U5 150.9 mm to (37.0, 112.0)
- moved H1 145.5 mm to (18.5, 14.0)
- moved C15 142.9 mm to (34.6, 104.2), turned to 0 degrees
- moved C9 132.3 mm to (40.9, 97.5), turned to 0 degrees
- moved H4 126.3 mm to (33.7, 133.5)
- moved U6 126.2 mm to (153.0, 15.5), turned to 90 degrees
- moved C16 115.3 mm to (152.0, 22.8), turned to 90 degrees
- moved R20 98.4 mm to (112.2, 30.5), turned to 270 degrees
- moved U12 98.0 mm to (150.0, 112.0)
- moved J21 89.0 mm to (108.0, 22.5), turned to 90 degrees
- moved U4 86.5 mm to (70.0, 32.0)
- moved C18 86.2 mm to (145.0, 12.5), turned to 90 degrees
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- renumbered C15 to C10, C12 to C11, C13 to C12, C19 to C13, C16 to C15, C17 to C16, C11 to C17, D2 to D1, H2 to H1, H3 to H2, H4 to H3, H5 to H4, H6 to H5, R15 to R14, R17 to R16, R18 to R17, R19 to R18, R20 to R19, R22 to R21, R23 to R22, R24 to R23, R25 to R24, R26 to R25, R27 to R26, R28 to R27, R29 to R28, R30 to R29, R31 to R30, R32 to R31, R7 to R6, R9 to R8, U14 to U11, U6 to U5, U10 to U9
Connections:
- C14 pad 1: /USBH_1 -> +3V3
- C14 pad 2: /USBH_1 -> GND
- C18 pad 1: +3V3 -> /IRQSTAT
- C18 pad 2: GND -> /PL2
- C19 pad 1: /IRQ1 -> +3V3
- C9 pad 1: +3V3 -> /IRQSTAT
- C9 pad 2: /PL2 -> /PL
- D1 pad 1: /MIN2_A -> /MIN1_A
- D1 pad 2: /MIN2_5 -> /MIN1_5
- D2 pad 1: +3V3 -> /MIN2_A
- D2 pad 2: /MIDI_RX1 -> /MIN2_5
- D3 pad 1: /TUNE_J -> GND
- D3 pad 2: /TUNE_N -> +3V3
- J11 pad 2: /CODEC_RST -> GND
- J11 pad 3: +5V -> /DISP_CS
- J11 pad 4: /MCLK -> /DISP_RST
- J11 pad 5: GND -> /DISP_DC
- J11 pad 6: /BCLK -> /MOSI1
- J11 pad 7: GND -> /SCK1
- J11 pad 8: /LRCLK -> +3V3
- J11 pad 9: GND -> (no net)
- J12 pad 1: +3V3 -> GND
- J12 pad 2: GND -> +3V3
- J12 pad 3: /DISP_CS -> /SDA
- J12 pad 4: /DISP_RST -> /SCL
- J13 pad 1: /MIN2_4 -> /MIN1_4
- J13 pad 2: /MIN2_5 -> /MIN1_5
- J14 pad 1: /MOUT5 -> /MIN2_4
- J14 pad 2: /MOUT4 -> /MIN2_5
- J14 pad 3: GND -> (no net)
- J15 pad 1: /MOUT2_5 -> /MOUT5
- J15 pad 2: /MOUT2_4 -> /MOUT4
- J16 pad 1: GND -> +12V
- J16 pad 2: +3V3 -> /CANH
- J16 pad 3: /SDA -> /CANL
- J16 pad 4: /SCL -> GND
- J17 pad 1: /TUNE_J -> +3V3
- J17 pad 2: GND -> /CODEC_RST
- J18 pad 1: (no net) -> /TUNE_J
- J18 pad 2: /TUNE_N -> GND
- J20 pad 1: /MIN1_4 -> GND
- J20 pad 2: /MIN1_5 -> /DLG2_TX
- J20 pad 3: (no net) -> /DLG2_RX
- J21 pad 1: /MCLK -> /CS9
- J21 pad 10: /I2SD6 -> /IRQ11
- J21 pad 11: GND -> /CS14
- J21 pad 12: GND -> /IRQ12
- J21 pad 13: GND -> /MISO
- J21 pad 2: /BCLK -> /IRQ7
- J21 pad 3: /LRCLK -> /CS10
- J21 pad 4: GND -> /IRQ8
- J21 pad 5: /I2SD1 -> /CS11
- J21 pad 6: /I2SD2 -> /IRQ9
- J21 pad 7: /I2SD3 -> /CS12
- J21 pad 8: /I2SD4 -> /IRQ10
- J21 pad 9: /I2SD5 -> /CS13
- J22 pad 1: +12V -> /MOUT2_5
- J22 pad 2: /CANH -> /MOUT2_4
- J22 pad 3: /CANL -> GND
- J23 pad 1: /CS1 -> /USBH_1
- J23 pad 10: /CS10 -> /USBH_5
- J23 pad 2: /CS2 -> /USBH_1
- J23 pad 3: /CS3 -> /USBH_2
- J23 pad 4: /CS4 -> /USBH_2
- J23 pad 5: /CS5 -> /USBH_3
- J23 pad 6: /CS6 -> /USBH_3
- J23 pad 7: /CS7 -> /USBH_4
- J23 pad 8: /CS8 -> /USBH_4
- J23 pad 9: /CS9 -> /USBH_5
- J24 pad 1: /CAN_TX -> /MCLK
- J24 pad 2: GND -> /BCLK
- J24 pad 3: +3V3 -> /LRCLK
- J24 pad 4: /CAN_RX -> GND
- J24 pad 5: (no net) -> /I2SD1
- J24 pad 6: /CANL -> /I2SD2
- J24 pad 7: /CANH -> /I2SD3
- J24 pad 8: /CAN_RS -> /I2SD4
- J25 pad 1: GND -> +5V
- J25 pad 2: /DLG2_TX -> GND
- R10 pad 1: +3V3 -> /MOUT_Y
- R10 pad 2: /MOUT4 -> /MOUT5
- R11 pad 1: /MOUT2_Y -> +3V3
- R11 pad 2: /MOUT2_5 -> /MOUT4
- R12 pad 1: /CAN_TRM -> /CANH
- R12 pad 2: /CANL -> /CAN_TRM
- R13 pad 1: /CANH -> /CAN_RS
- R13 pad 2: /CAN_TRM -> GND
- R14 pad 1: /TUNE_N -> /TUNE_J
- R14 pad 2: GND -> /TUNE_N
- R15 pad 1: +3V3 -> /TUNE_N
- R16 pad 1: /XMOSI0 -> /XSCLK0
- R16 pad 2: /XMOSI -> /XSCLK
- R17 pad 1: /XLDAC0 -> /XMOSI0
- R17 pad 2: /XLDAC -> /XMOSI
- R18 pad 1: /XCONVST0 -> /XLDAC0
- R18 pad 2: /XCONVST -> /XLDAC
- R19 pad 1: /XRST0 -> /XCONVST0
- R19 pad 2: /XRST -> /XCONVST
- R20 pad 1: /MIN1_4 -> /XRST0
- R20 pad 2: /MIN1_A -> /XRST
- R21 pad 1: /IRQ2 -> /IRQ1
- R22 pad 1: /IRQ3 -> /IRQ2
- R23 pad 1: /IRQ4 -> /IRQ3
- R24 pad 1: /IRQ5 -> /IRQ4
- R25 pad 1: /IRQ6 -> /IRQ5
- R26 pad 1: /IRQ7 -> /IRQ6
- R27 pad 1: /IRQ8 -> /IRQ7
- R28 pad 1: /IRQ9 -> /IRQ8
- R29 pad 1: /IRQ10 -> /IRQ9
- R30 pad 1: /IRQ11 -> /IRQ10
- R31 pad 1: /IRQ12 -> /IRQ11
- R32 pad 1: /XSCLK0 -> /IRQ12
- R32 pad 2: /XSCLK -> GND
- R33 pad 1: /IRQSTAT -> +3V3
- R34 pad 1: +3V3 -> /MOUT2_Y
- R34 pad 2: /MOUT2_4 -> /MOUT2_5
- R35 pad 1: /CAN_RS -> +3V3
- R35 pad 2: GND -> /MOUT2_4
- R5 pad 1: /IRQSTAT -> +3V3
- R6 pad 1: /MIN2_4 -> /MIN1_4
- R6 pad 2: /MIN2_A -> /MIN1_A
- R7 pad 1: /MIN1_A -> /MIN2_4
- R7 pad 2: /MIN1_5 -> /MIN2_A
- R8 pad 2: /MIDI_RX2 -> /MIDI_RX1
- R9 pad 1: /MOUT_Y -> +3V3
- R9 pad 2: /MOUT5 -> /MIDI_RX2
- U10 pad 1: (no net) -> /MIN2_A
- U10 pad 2: /MIDI_TX -> /MIN2_5
- U10 pad 3: GND -> (no net)
- U10 pad 4: /MOUT_Y -> /MIDI_RX2
- U10 pad 5: +3V3 -> GND
- U11 pad 2: /MIDI_TX2 -> /MIDI_TX
- U11 pad 4: /MOUT2_Y -> /MOUT_Y
- U12 pad 1: /MIN1_A -> /CAN_TX
- U12 pad 2: /MIN1_5 -> GND
- U12 pad 3: (no net) -> +3V3
- U12 pad 4: /MIDI_RX1 -> /CAN_RX
- U12 pad 5: GND -> (no net)
- U12 pad 6: +3V3 -> /CANL
- U13 pad 1: GND -> (no net)
- U13 pad 2: +3V3 -> /TUNE_N
- U13 pad 3: /TUNE_N -> GND
- U14 pad 1: +3V3 -> (no net)
- U14 pad 2: /PL -> /MIDI_TX2
- U4 pad 1: /PL -> /CS1
- U4 pad 10: /CHAIN -> /CS10
- U4 pad 11: /IRQ4 -> /CS11
- U4 pad 12: /IRQ3 -> GND
- U4 pad 13: /IRQ2 -> /CS12
- U4 pad 14: /IRQ1 -> /CS13
- U4 pad 15: GND -> /CS14
- U4 pad 16: +3V3 -> /IRQSTAT
- U4 pad 2: /SCLK -> /CS2
- U4 pad 3: GND -> /CS3
- U4 pad 4: GND -> /CS4
- U4 pad 5: /IRQ6 -> /CS5
- U4 pad 6: /IRQ5 -> /CS6
- U4 pad 7: (no net) -> /CS7
- U4 pad 8: GND -> /CS8
- U4 pad 9: /Q7A -> /CS9
- U5 pad 1: /PL2 -> /PL
- U5 pad 10: GND -> /CHAIN
- U5 pad 11: GND -> /IRQ4
- U5 pad 12: GND -> /IRQ3
- U5 pad 13: /IRQ12 -> /IRQ2
- U5 pad 14: /IRQ11 -> /IRQ1
- U5 pad 3: /IRQ10 -> GND
- U5 pad 4: /IRQ9 -> GND
- U5 pad 5: /IRQ8 -> /IRQ6
- U5 pad 6: /IRQ7 -> /IRQ5
- U5 pad 9: /CHAIN -> /Q7A
- U6 pad 1: /IRQSTAT -> /PL2
- U6 pad 2: /Q7A -> /SCLK
- U6 pad 3: GND -> /IRQ10
- U6 pad 4: /MISO -> /IRQ9
- U6 pad 5: +3V3 -> /IRQ8
- U7 pad 1: +3V3 -> /IRQSTAT
- U7 pad 2: /SCLK -> /Q7A
- U7 pad 3: /MOSI -> GND
- U7 pad 4: /LDAC -> /MISO
- U7 pad 5: /CONVST -> +3V3
- U8 pad 1: /CS9 -> +3V3
- U8 pad 10: /IRQ11 -> GND
- U8 pad 11: /CS14 -> (no net)
- U8 pad 12: /IRQ12 -> (no net)
- U8 pad 13: /MISO -> (no net)
- U8 pad 14: GND -> /XRST0
- U8 pad 15: /XSCLK -> /XCONVST0
- U8 pad 16: GND -> /XLDAC0
- U8 pad 17: /XMOSI -> /XMOSI0
- U8 pad 18: GND -> /XSCLK0
- U8 pad 19: /XLDAC -> GND
- U8 pad 2: /IRQ7 -> /SCLK
- U8 pad 20: GND -> +3V3
- U8 pad 3: /CS10 -> /MOSI
- U8 pad 4: /IRQ8 -> /LDAC
- U8 pad 5: /CS11 -> /CONVST
- U8 pad 6: /IRQ9 -> /SPARE2
- U8 pad 7: /CS12 -> GND
- U8 pad 8: /IRQ10 -> GND
- U8 pad 9: /CS13 -> GND
- U9 pad 1: /MIN2_A -> /MIN1_A
- U9 pad 2: /MIN2_5 -> /MIN1_5
- U9 pad 4: /MIDI_RX2 -> /MIDI_RX1
Routing:
- net GND: track 1599.1 -> 1602.8 mm
Other:
- board text added: "musicbrain.nl/hw/busboard rev 3.1 - gen 2: 6x slot 2x12 + audio, 16xCS/12xIRQ, MIDI 2x2, USB-host"
- board text removed: "musicbrain.nl/hw/busboard rev 3.0 - gen 2: 6x slot 2x12 + audio, 16xCS/12xIRQ, MIDI 2x2, USB-host"
Changed lines of the file:
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@@
     (title "MusicBrain SPI-busboard")
     (date "2026-07-16")
-    (rev "3.0")
+    (rev "3.1")
     (company "MusicBrain project")
   )
@@
     )
   )
+  (footprint "Connector_PinHeader_2.54mm:PinHeader_1x02_P2.54mm_Vertical"
+    (at 66.3 129.19 180)
+    (layer "F.Cu")
+    (descr "Through hole straight pin header, 1x02, 2.54mm pitch, single row")
+    (tags "Through hole pin header THT 1x02 2.54mm single row")
+    (property "Reference" "J25"
+      (at -2.6 1.27 0)
+      (layer "F.SilkS")
+      (effects
+        (font
+          (size 1 1)
+          (thickness 0.15)
+        )
+      )
+    )
+    (property "Value" "AXON +5V"
+      (at 0 4.92 0)
+      (layer "F.Fab")
+      (effects
+        (font
+          (size 1 1)
+          (thickness 0.15)
+        )
+      )
+    )
+    (attr through_hole)
+    (fp_line
+      (start -1.38 -1.38)
+      (end 0 -1.38)
+      (stroke
+        (width 0.12)
+        (type solid)
+      )
+      (layer "F.SilkS")
+    )
+    (fp_line
+      (start -1.38 0)
+      (end -1.38 -1.38)
+      (stroke
+        (width 0.12)
+        (type solid)
+      )
+      (layer "F.SilkS")
+    )
+    (fp_line
+      (start -1.38 1.27)
+      (end -1.38 3.92)
+      (stroke
+        (width 0.12)
+        (type solid)
+      )
+      (layer "F.SilkS")
+    )
+    (fp_line
+      (start -1.38 1.27)
+      (end 1.38 1.27)
+      (stroke
+        (width 0.12)
+        (type solid)
+      )
+      (layer "F.SilkS")
+    )
+    (fp_line
+      (start -1.38 3.92)
+      (end 1.38 3.92)
+      (stroke
+        (width 0.12)
+        (type solid)
+      )
+      (layer "F.SilkS")
+    )
+    (fp_line
+      (start 1.38 1.27)
+      (end 1.38 3.92)
+      (stroke
+        (width 0.12)
+        (type solid)
+      )
+      (layer "F.SilkS")
+    )
+    (fp_rect
+      (start -1.77 -1.77)
+      (end 1.77 4.32)
+      (stroke
+        (width 0.05)
+        (type solid)
+      )
+      (fill no)
+      (layer "F.CrtYd")
+    )
+    (fp_line
+      (start -1.27 -0.635)
+      (end -0.635 -1.27)
+      (stroke
+        (width 0.1)
+        (type solid)
+      )
+      (layer "F.Fab")
+    )
+    (fp_line
+      (start -1.27 3.81)
+      (end -1.27 -0.635)
+      (stroke
+        (width 0.1)
+        (type solid)
+      )
+      (layer "F.Fab")
+    )
+    (fp_line
+      (start -0.635 -1.27)
+      (end 1.27 -1.27)
+      (stroke
+        (width 0.1)
+        (type solid)
+      )
+      (layer "F.Fab")
+    )
+    (fp_line
+      (start 1.27 -1.27)
+      (end 1.27 3.81)
+      (stroke
+        (width 0.1)
+        (type solid)
+      )
+      (layer "F.Fab")
+    )
+    (fp_line
+      (start 1.27 3.81)
+      (end -1.27 3.81)
+      (stroke
+        (width 0.1)
+        (type solid)
+      )
+      (layer "F.Fab")
+    )
+    (fp_text user "${REFERENCE}"
+      (at 0 1.27 90)
+      (layer "F.Fab")
+      (effects
+        (font
+          (size 1 1)
+          (thickness 0.15)
+        )
+      )
+    )
+    (pad "1" thru_hole rect
+      (at 0 0 180)
+      (size 1.7 1.7)
+      (drill 1)
+      (layers "*.Cu" "*.Mask")
+      (remove_unused_layers no)
+      (net 2 "+5V")
+    )
+    (pad "2" thru_hole circle
+      (at 0 2.54 180)
+      (size 1.7 1.7)
+      (drill 1)
+      (layers "*.Cu" "*.Mask")
+      (remove_unused_layers no)
+      (net 5 "GND")
+    )
+    (model "${KICAD10_3DMODEL_DIR}/Connector_PinHeader_2.54mm.3dshapes/PinHeader_1x02_P2.54mm_Vertical.step"
+      (offset
+        (xyz 0 0 0)
+      )
+      (scale
+        (xyz 1 1 1)
+      )
+      (rotate
+        (xyz 0 0 0)
+      )
+    )
+  )
   (footprint "Connector_PinHeader_2.54mm:PinHeader_1x04_P2.54mm_Vertical"
     (at 71.5 135 90)
@@
     )
   )
+  (segment (start 66.3 126.65) (end 70 126.65) (width 0.25) (layer "F.Cu") (net 5))
   (segment (start 59.3034 55.8789) (end 59.3034 62.6734) (width 0.35) (layer "F.Cu") (net 1))
   (segment (start 59.3034 62.6734) (end 61.99 65.36) (width 0.35) (layer "F.Cu") (net 1))
@@
     (stroke (width 0.1) (type default)) (fill none)
     (layer "Edge.Cuts"))
-  (gr_text "musicbrain.nl/hw/busboard rev 3.0 - gen 2: 6x slot 2x12 + audio, 16xCS/12xIRQ, MIDI 2x2, USB-host" (at 116.6 98.5 0) (layer "F.SilkS")
+  (gr_text "musicbrain.nl/hw/busboard rev 3.1 - gen 2: 6x slot 2x12 + audio, 16xCS/12xIRQ, MIDI 2x2, USB-host" (at 116.6 98.5 0) (layer "F.SilkS")
     (effects (font (size 1.5 1.5) (thickness 0.25))))
   (zone (net 5) (net_name "GND") (layer "F.Cu")
