File: hardware/schematics/musicbrain-axon/musicbrain-axon.kicad_pcb (KiCad board)
At the start: 2 copper layers, 70 x 45 mm, 52 parts, among them J1 BUSBOARD, J2 USB-C, J3 MAGJACK, J4 DEBUG, SW1 RESET, SW2 BOOT, U1 ESP32-S3-WROOM-1U-N8R2, U2 W5500, U3 AMS1117-3.3, Y1 25MHz

Commit message: Axon: J4 (debug-UART) naar de noordrand — korte route (DRC 0/0), weg van de Teensy-zone; silk herschikt
Co-Authored-By: Claude Fable 5 <noreply@anthropic.com>
Parts:
- moved J4 43.2 mm to (136.0, 101.8), turned to 0 degrees
Routing:
- net /DBG_RX: track 40.9 -> 9.92 mm
- net /DBG_TX: track 38.1 -> 15.6 mm, vias 0 -> 1
- net +3V3: track 154.4 -> 138.4 mm, vias 7 -> 5
- net +3V3A: track 88.0 -> 74.5 mm, vias 7 -> 0
- net /W_INT: track 45.1 -> 32.1 mm
- net /ESP_EN: track 49.1 -> 61.6 mm, vias 4 -> 2
- net /W_MISO: track 26.7 -> 37.7 mm
- net GND: track 412.4 -> 422.8 mm, vias 26 -> 25
- net /TXN: track 27.2 -> 35.4 mm, vias 1 -> 2
- net /XO: track 17.9 -> 13.3 mm, vias 3 -> 1
- net /LINK_K: track 31.0 -> 26.8 mm
- net /LINKLED: track 17.9 -> 21.9 mm, vias 2 -> 0
- net /W_CS: track 31.1 -> 34.3 mm
- net /W_RST: track 30.0 -> 27.1 mm
- net /AXON_RX: track 36.9 -> 39.7 mm
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Other:
- board text added: "MUSICBRAIN AXON"
- board text added: "musicbrain.nl/hw/axon (0.1)"
- board text removed: "MUSICBRAIN AXON rev 0.1"
- board text removed: "musicbrain.nl/hw/axon"

Commit message: Axon J1: alle 6 pinnen, 2+4 gegroepeerd (5V/GND->J25, GND/RX/TX/GND->J19)
RX op pin 4, TX op pin 5: beide kabels recht 1:1 (UART-kruising in de
pinvolgorde). Per-pin silk-labels uitgelijnd onder de pads (0.8mm-font,
silk-helper met optionele grootte). Geroute DRC 0/0; kabeltabel in README.

Co-Authored-By: Claude Fable 5 <noreply@anthropic.com>
Connections:
- J1 pad 3: /AXON_TX -> GND
- J1 pad 5: GND -> /AXON_TX
- J1 pad 6: (no net) -> GND
Routing:
- net /RXN: track 15.7 -> 38.1 mm, vias 2 -> 0
- net /ESP_EN: track 61.6 -> 48.1 mm
- net /W_RST: track 27.1 -> 37.0 mm
- net /XI: track 12.9 -> 21.8 mm
- net /W_SCLK: track 29.6 -> 37.3 mm
- net /TXN: track 35.4 -> 27.9 mm, vias 2 -> 3
- net /W_MISO: track 37.7 -> 30.4 mm
- net /W_MOSI: track 30.9 -> 38.0 mm
- net /XO: track 13.3 -> 20.1 mm, vias 1 -> 3
- net +3V3: track 138.4 -> 132.7 mm, vias 5 -> 2
- net /LINKLED: track 21.9 -> 16.3 mm
- net /AXON_TX: track 37.3 -> 41.7 mm
- net /ACT_K: track 35.7 -> 31.3 mm
- net GND: track 422.8 -> 426.2 mm, vias 25 -> 28
- net /W_CS: track 34.3 -> 37.2 mm
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Other:
- board text added: "5V"
- board text added: "GND"
- board text added: "RX"
- board text added: "TX"
- board text removed: "5V GND TX RX GND -"
