File: hardware/schematics/musicbrain-vcf8kern/musicbrain-vcf8kern.kicad_pcb (KiCad board)
At the start: 4 copper layers, 110 x 92 mm, 412 parts, among them J1 KERNSLOT, J2 AUDIO IN, J3 AUDIO UIT, Q1 2N7002, U1 SSI2140, U11 74HC4051, U12 74HC4051, U13 74HC4051, U14 74HC4051, U15 74HC4051, U16 74HC4051, U17 74HC4051, U18 74HC4051, U2 SSI2140, U21 TL074, U22 TL074, U23 TL074, U24 TL074, U25 TL074, U3 SSI2140, U31 AD5754BREZ, U32 AD5754BREZ, U33 ADR421, U34 DAC128S085CIMTX, U35 74HC4051, U36 LM311, U4 SSI2140, U5 SSI2140, U6 SSI2140, U7 SSI2140, U8 SSI2140

Commit message: VCF8-kern rev 0.1: fab + website (component/release cortex-v0.3)
Bord af en reproduceerbaar (generator + DRC 0/0 op macOS). Toegevoegd:
- fab-pakket (BOM + CPL; gerbers/zip blijven ge-ignored, regenereerbaar)
- website-assets: beschrijving.txt, aansluitoverzicht (SVG + json),
  widget.json (3D + hotspots), pinouts J1/J2/J3, README-aansluitsectie
- gepubliceerd naar de lokale Imprint-site als component vcf8kern@v0.1 en
  gepind in release cortex-v0.3 (publish_release.py PINS + product)

Scripts cross-platform (macOS + Windows), net als cardlib.py:
- nieuwe kicadcli.py-helper (autodetect kicad-cli) gebruikt door
  board_overview.py, publish_board.py, widget_export.py
- make_fab.sh: ROOT uit scriptlocatie, kicad-cli/python autodetect

Co-Authored-By: Claude Opus 4.8 <noreply@anthropic.com>
Routing:
- net AOUT3: track 19.2 -> 74.7 mm
- net GND: track 1580.8 -> 1605.1 mm, vias 244 -> 254
- net CS2: track 118.1 -> 132.3 mm, vias 10 -> 8
- net IN12: track 14.7 -> 12.0 mm
- net MODE1: track 314.9 -> 316.8 mm
- net MOUT7: track 16.8 -> 18.7 mm, vias 0 -> 2
- net MODE0: track 342.9 -> 344.6 mm
- net MN8_7: track 28.4 -> 29.4 mm
- net +3V3: track 386.5 -> 387.1 mm
